File: BGP_V1/BUF/BUF.sch (KiCad schematic (older format))
At the start: 23 parts, among them P1 CONN_01X05, P2 CONN_01X02, P3 CONN_01X12, U1 MC33178, U2 TLV170

Commit message: Concentric pot fixups for 1_BUF
Connections:
- net VF1_1: now also P3.1 (P1), P3.2 (P2); no longer P3.7 (P7)
- net VF1_2: now also P3.3 (P3), P3.4 (P4), P3.5 (P5); no longer P3.10 (P10), P3.8 (P8), P3.9 (P9)
- net VF2_2: now also P3.6 (P6); no longer P3.11 (P11), P3.12 (P12)
- net VP1_1: now also P3.7 (P7), P3.8 (P8); no longer P3.1 (P1)
- net VP1_2: now also P3.9 (P9); no longer P3.2 (P2), P3.3 (P3)
- net VP2_1: now also P3.10 (P10), P3.11 (P11); no longer P3.4 (P4)
- net VP2_2: now also P3.12 (P12); no longer P3.5 (P5), P3.6 (P6)
Changed lines of the file:
@@
 EESchema Schematic File Version 2
-LIBS:BUF-rescue
 LIBS:power
 LIBS:device
@@
 $EndComp
 $Comp
-L Earth #PWR8
+L Earth #PWR01
 U 1 1 5A4D6930
 P 7450 4150
-F 0 "#PWR8" H 7450 3900 50  0001 C CNN
+F 0 "#PWR01" H 7450 3900 50  0001 C CNN
 F 1 "Earth" H 7450 4000 50  0001 C CNN
 F 2 "" H 7450 4150 50  0000 C CNN
@@
 V-
 $Comp
-L Earth #PWR6
+L Earth #PWR02
 U 1 1 5A4D7443
 P 5850 4100
-F 0 "#PWR6" H 5850 3850 50  0001 C CNN
+F 0 "#PWR02" H 5850 3850 50  0001 C CNN
 F 1 "Earth" H 5850 3950 50  0001 C CNN
 F 2 "" H 5850 4100 50  0000 C CNN
@@
 $EndComp
 $Comp
-L Earth #PWR7
+L Earth #PWR03
 U 1 1 5A4D75B6
 P 6450 4650
-F 0 "#PWR7" H 6450 4400 50  0001 C CNN
+F 0 "#PWR03" H 6450 4400 50  0001 C CNN
 F 1 "Earth" H 6450 4500 50  0001 C CNN
 F 2 "" H 6450 4650 50  0000 C CNN
@@
 V+
 $Comp
-L Earth #PWR1
+L Earth #PWR04
 U 1 1 5A4D8532
 P 2550 3800
-F 0 "#PWR1" H 2550 3550 50  0001 C CNN
+F 0 "#PWR04" H 2550 3550 50  0001 C CNN
 F 1 "Earth" H 2550 3650 50  0001 C CNN
 F 2 "" H 2550 3800 50  0000 C CNN
@@
 $EndComp
 $Comp
-L Earth #PWR2
+L Earth #PWR05
 U 1 1 5A4D8B77
 P 2550 4300
-F 0 "#PWR2" H 2550 4050 50  0001 C CNN
+F 0 "#PWR05" H 2550 4050 50  0001 C CNN
 F 1 "Earth" H 2550 4150 50  0001 C CNN
 F 2 "" H 2550 4300 50  0000 C CNN
@@
 	1    0    0    -1
 $EndComp
-Text Label 9600 3250 2    60   ~ 0
+Text Label 9600 3950 2    60   ~ 0
 VP1_1
+Text Label 9600 4050 2    60   ~ 0
+VP1_2
+Text Label 9600 4250 2    60   ~ 0
+VP2_1
+Text Label 9600 4350 2    60   ~ 0
+VP2_2
 Text Label 9600 3350 2    60   ~ 0
-VP1_2
-Text Label 9600 3550 2    60   ~ 0
-VP2_1
+VF1_1
+Text Label 9600 3450 2    60   ~ 0
+VF1_2
 Text Label 9600 3650 2    60   ~ 0
-VP2_2
-Text Label 9600 3850 2    60   ~ 0
-VF1_1
-Text Label 9600 3950 2    60   ~ 0
-VF1_2
-Text Label 9600 4150 2    60   ~ 0
 VF2_1
-Text Label 9600 4250 2    60   ~ 0
+Text Label 9600 3750 2    60   ~ 0
 VF2_2
 $Comp
@@
 $EndComp
 $Comp
-L Earth #PWR3
+L Earth #PWR06
 U 1 1 5A52D771
 P 3300 4150
-F 0 "#PWR3" H 3300 3900 50  0001 C CNN
+F 0 "#PWR06" H 3300 3900 50  0001 C CNN
 F 1 "Earth" H 3300 4000 50  0001 C CNN
 F 2 "" H 3300 4150 50  0000 C CNN
@@
 $EndComp
 $Comp
-L Earth #PWR4
+L Earth #PWR07
 U 1 1 5A52D7C1
 P 3650 4150
-F 0 "#PWR4" H 3650 3900 50  0001 C CNN
+F 0 "#PWR07" H 3650 3900 50  0001 C CNN
 F 1 "Earth" H 3650 4000 50  0001 C CNN
 F 2 "" H 3650 4150 50  0000 C CNN
@@
 $EndComp
 $Comp
-L Earth #PWR5
+L Earth #PWR08
 U 1 1 5A52E514
 P 4650 4150
-F 0 "#PWR5" H 4650 3900 50  0001 C CNN
+F 0 "#PWR08" H 4650 3900 50  0001 C CNN
 F 1 "Earth" H 4650 4000 50  0001 C CNN
 F 2 "" H 4650 4150 50  0000 C CNN
@@
 Wire Wire Line
 	8900 3950 8850 3950
-Wire Wire Line
-	9600 4250 9600 4350
-Wire Wire Line
-	9600 4050 9600 3950
-Wire Wire Line
-	9600 3650 9600 3750
-Wire Wire Line
-	9600 3450 9600 3350
 Wire Wire Line
 	7100 3850 7200 3850
@@
 	1    0    0    -1
 $EndComp
+Wire Wire Line
+	9600 4150 9600 4250
+Wire Wire Line
+	9600 3850 9600 3950
+Wire Wire Line
+	9600 3550 9600 3650
+Wire Wire Line
+	9600 3250 9600 3350
 $EndSCHEMATC

Commit message: BOM for V1 BGP
Parts:
- C2, C5: footprint Capacitors_SMD:C_1206_HandSoldering -> Capacitors_Tantalum_SMD:TantalC_SizeS_EIA-3216
- C6: footprint Capacitors_SMD:C_1206_HandSoldering -> Capacitors_SMD:C_0805_HandSoldering
Changed lines of the file:
@@
 F 0 "C5" H 8760 4020 50  0000 L CNN
 F 1 "10u" H 8760 3870 50  0000 L CNN
-F 2 "Capacitors_SMD:C_1206_HandSoldering" H 8750 3950 50  0001 C CNN
+F 2 "Capacitors_Tantalum_SMD:TantalC_SizeS_EIA-3216" H 8750 3950 50  0001 C CNN
 F 3 "" H 8750 3950 50  0000 C CNN
 	1    8750 3950
@@
 F 0 "C6" H 9010 4420 50  0000 L CNN
 F 1 "10u" H 9010 4270 50  0000 L CNN
-F 2 "Capacitors_SMD:C_1206_HandSoldering" H 9000 4350 50  0001 C CNN
+F 2 "Capacitors_SMD:C_0805_HandSoldering" H 9000 4350 50  0001 C CNN
 F 3 "" H 9000 4350 50  0000 C CNN
 	1    9000 4350
@@
 F 0 "C2" H 4560 3820 50  0000 L CNN
 F 1 "10u" H 4560 3670 50  0000 L CNN
-F 2 "Capacitors_SMD:C_1206_HandSoldering" H 4550 3750 50  0001 C CNN
+F 2 "Capacitors_Tantalum_SMD:TantalC_SizeS_EIA-3216" H 4550 3750 50  0001 C CNN
 F 3 "" H 4550 3750 50  0000 C CNN
 	1    4550 3750
