File: BGP_V0/VOL/VOL.sch (KiCad schematic (older format))
At the start: 23 parts, among them IC1 TC7660SO-08, P1 CONN_01X05, P2 CONN_01X03, P3 CONN_01X05, P4 CONN_01X05, P5 CONN_01X02

Commit message: Pot fixups for silkscreen overlap
Parts:
- RV1: footprint Potentiometers:Potentiometer_Alps_RK097_Single_Vertical -> LIBS:Potentiometer_Alps_RK097_Single_Vertical
Changed lines of the file:
@@
 F 0 "RV1" H 5000 4420 50  0000 C CNN
 F 1 "POT" H 5000 4500 50  0000 C CNN
-F 2 "Potentiometers:Potentiometer_Alps_RK097_Single_Vertical" H 5000 4500 50  0001 C CNN
+F 2 "LIBS:Potentiometer_Alps_RK097_Single_Vertical" H 5000 4500 50  0001 C CNN
 F 3 "" H 5000 4500 50  0000 C CNN
 	1    5000 4500

Commit message: V_0 Updates for caps, gerbers updated
Parts:
- C1: footprint Capacitors_SMD:C_1206_HandSoldering -> Capacitors_Tantalum_SMD:TantalC_SizeR_EIA-2012
- C2, C4: footprint Capacitors_SMD:C_0603_HandSoldering -> Capacitors_SMD:C_0805_HandSoldering
- C5: footprint Capacitors_SMD:C_1206_HandSoldering -> Capacitors_SMD:C_0805_HandSoldering
Changed lines of the file:
@@
 F 0 "C1" H 4810 4270 50  0000 L CNN
 F 1 "22u" H 4810 4120 50  0000 L CNN
-F 2 "Capacitors_SMD:C_1206_HandSoldering" H 4800 4200 50  0001 C CNN
+F 2 "Capacitors_Tantalum_SMD:TantalC_SizeR_EIA-2012" H 4800 4200 50  0001 C CNN
 F 3 "" H 4800 4200 50  0000 C CNN
 	1    4800 4200
@@
 F 0 "C5" H 6210 2770 50  0000 L CNN
 F 1 "22u" H 6210 2620 50  0000 L CNN
-F 2 "Capacitors_SMD:C_1206_HandSoldering" H 6200 2700 50  0001 C CNN
+F 2 "Capacitors_SMD:C_0805_HandSoldering" H 6200 2700 50  0001 C CNN
 F 3 "" H 6200 2700 50  0000 C CNN
 	1    6200 2700
@@
 F 0 "C4" H 5810 3470 50  0000 L CNN
 F 1 "1u" H 5810 3320 50  0000 L CNN
-F 2 "Capacitors_SMD:C_0603_HandSoldering" H 5800 3400 50  0001 C CNN
+F 2 "Capacitors_SMD:C_0805_HandSoldering" H 5800 3400 50  0001 C CNN
 F 3 "" H 5800 3400 50  0000 C CNN
 	1    5800 3400
@@
 F 0 "C2" H 4210 3220 50  0000 L CNN
 F 1 "1u" H 4210 3070 50  0000 L CNN
-F 2 "Capacitors_SMD:C_0603_HandSoldering" H 4200 3150 50  0001 C CNN
+F 2 "Capacitors_SMD:C_0805_HandSoldering" H 4200 3150 50  0001 C CNN
 F 3 "" H 4200 3150 50  0000 C CNN
 	1    4200 3150
