File: BGP_V1/VOL/VOL.kicad_pcb (KiCad board)
At the start: 2 copper layers, 60 x 30 mm, 33 parts, among them IC1 TC7660SO-08, P1 CONN_01X03, P2 CONN_01X02, P3 CONN_01X05, P4 CONN_01X05, P5 CONN_01X05, P6 Conn_01x14, P7 CONN_02X02, U1 OPA2170

Commit message: Slight changes to Port layer placement - gerbers done
Other:
- board text added: "+"
- board text added: "-"
- board text added: "B"
- board text added: "B+"
- board text added: "B-"
- board text added: "BRIDGE"
- board text added: "G"
- board text added: "HPF"
- board text added: "I"
- board text added: "N"
- board text added: "NECK"
- board text added: "O"
Changed lines of the file:
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@@
     (area 118.924999 80.424999 179.303001 112.85588)
     (thickness 1.6)
-    (drawings 9)
+    (drawings 34)
     (tracks 241)
     (zones 0)
@@
     (at 177.2 107.5 180)
     (descr "3-way 2.54mm pitch terminal block, Phoenix MPT series")
-    (fp_text reference P1 (at -0.8 3.8 180) (layer B.SilkS)
+    (fp_text reference P1 (at -0.1 5 180) (layer B.SilkS)
       (effects (font (size 0.6 0.6) (thickness 0.15)) (justify mirror))
     )
@@
     (at 168.4 107.5 180)
     (descr "2-way 2.54mm pitch terminal block, Phoenix MPT series")
-    (fp_text reference P2 (at -1 3.8 180) (layer B.SilkS)
+    (fp_text reference P2 (at -0.1 5 180) (layer B.SilkS)
       (effects (font (size 0.6 0.6) (thickness 0.15)) (justify mirror))
     )
@@
     )
   )
+  (gr_text B- (at 177.2 103.6) (layer B.SilkS)
+    (effects (font (size 0.6 0.6) (thickness 0.15)) (justify mirror))
+  )
+  (gr_text O (at 174.7 103.6) (layer B.SilkS)
+    (effects (font (size 0.6 0.6) (thickness 0.15)) (justify mirror))
+  )
+  (gr_text G (at 172.1 103.6) (layer B.SilkS)
+    (effects (font (size 0.6 0.6) (thickness 0.15)) (justify mirror))
+  )
+  (gr_text B- (at 165.8 103.6) (layer B.SilkS)
+    (effects (font (size 0.6 0.6) (thickness 0.15)) (justify mirror))
+  )
+  (gr_text B+ (at 168.4 103.6) (layer B.SilkS)
+    (effects (font (size 0.6 0.6) (thickness 0.15)) (justify mirror))
+  )
+  (gr_text B (at 155.4 108) (layer B.SilkS)
+    (effects (font (size 0.6 0.6) (thickness 0.15)) (justify mirror))
+  )
+  (gr_text N (at 157.4 108) (layer B.SilkS)
+    (effects (font (size 0.6 0.6) (thickness 0.15)) (justify mirror))
+  )
+  (gr_text - (at 140.9 103.6) (layer B.SilkS)
+    (effects (font (size 0.6 0.6) (thickness 0.15)) (justify mirror))
+  )
+  (gr_text G (at 140.9 101.6) (layer B.SilkS)
+    (effects (font (size 0.6 0.6) (thickness 0.15)) (justify mirror))
+  )
+  (gr_text O (at 140.9 107.6) (layer B.SilkS)
+    (effects (font (size 0.6 0.6) (thickness 0.15)) (justify mirror))
+  )
+  (gr_text I (at 140.9 105.6) (layer B.SilkS)
+    (effects (font (size 0.6 0.6) (thickness 0.15)) (justify mirror))
+  )
+  (gr_text + (at 141 99.6) (layer B.SilkS)
+    (effects (font (size 0.6 0.6) (thickness 0.15)) (justify mirror))
+  )
+  (gr_text - (at 130.9 103.5) (layer B.SilkS)
+    (effects (font (size 0.6 0.6) (thickness 0.15)) (justify mirror))
+  )
+  (gr_text G (at 130.9 101.5) (layer B.SilkS)
+    (effects (font (size 0.6 0.6) (thickness 0.15)) (justify mirror))
+  )
+  (gr_text O (at 130.9 107.5) (layer B.SilkS)
+    (effects (font (size 0.6 0.6) (thickness 0.15)) (justify mirror))
+  )
+  (gr_text I (at 130.9 105.5) (layer B.SilkS)
+    (effects (font (size 0.6 0.6) (thickness 0.15)) (justify mirror))
+  )
+  (gr_text + (at 131 99.5) (layer B.SilkS)
+    (effects (font (size 0.6 0.6) (thickness 0.15)) (justify mirror))
+  )
+  (gr_text O (at 120.9 107.6) (layer B.SilkS)
+    (effects (font (size 0.6 0.6) (thickness 0.15)) (justify mirror))
+  )
+  (gr_text I (at 120.9 105.6) (layer B.SilkS)
+    (effects (font (size 0.6 0.6) (thickness 0.15)) (justify mirror))
+  )
+  (gr_text - (at 120.9 103.6) (layer B.SilkS)
+    (effects (font (size 0.6 0.6) (thickness 0.15)) (justify mirror))
+  )
+  (gr_text G (at 120.9 101.6) (layer B.SilkS)
+    (effects (font (size 0.6 0.6) (thickness 0.15)) (justify mirror))
+  )
+  (gr_text + (at 121 99.6) (layer B.SilkS)
+    (effects (font (size 0.6 0.6) (thickness 0.15)) (justify mirror))
+  )
+  (gr_text NECK (at 143.9 96.8) (layer B.SilkS)
+    (effects (font (size 0.6 0.6) (thickness 0.15)) (justify mirror))
+  )
+  (gr_text BRIDGE (at 133.6 96.8) (layer B.SilkS)
+    (effects (font (size 0.6 0.6) (thickness 0.15)))
+  )
+  (gr_text HPF (at 123.9 96.9) (layer B.SilkS)
+    (effects (font (size 0.6 0.6) (thickness 0.15)))
+  )
   (gr_text "BGP V1.0\nVolume / Power" (at 130.8 82.5) (layer B.SilkS)

Commit message: Error found/corrected in 1_VOL. Modified to use ALPS RK097 dual shaft, quad gang.
Parts:
- added R11: 11k, Resistors_SMD:R_0603_HandSoldering, B.Cu at (165.3, 84.0)
- added R12: 11k, Resistors_SMD:R_0603_HandSoldering, B.Cu at (165.3, 86.5)
- P6: value Conn_01x14 -> CONN_01X12; footprint LIBS:Potentiometer_TT_P08X_Quad_Vertical_Dual_Shaft -> LIBS:Potentiometer_Alps_RK097_Quad_Vertical_Dual_Shaft
- R10: value 22k -> 11k
- R9: value 18k -> 8.45k
- moved P6 1.63 mm to (175.4, 84.0)
- moved R9 0.58 mm to (166.6, 87.1)
Connections:
- P1 pad 1: /BAT- -> Earth
- P1 pad 3: Earth -> /BAT-
- P6 pad 1: Net-(P6-Pad1) -> Earth
- P6 pad 10: /VB2_3 -> Earth
- P6 pad 11: Earth -> /OUT
- P6 pad 12: /OUT_N -> /VP_1
- P6 pad 2: Net-(P6-Pad2) -> /VB1_2
- P6 pad 3: Net-(P6-Pad3) -> /OUT_B
- P6 pad 5: /VP_OUT -> /VB2_2
- P6 pad 6: /VP_1 -> /OUT_N
- P6 pad 7: /VB1_3 -> Net-(P6-Pad7)
- P6 pad 8: Earth -> Net-(P6-Pad8)
- P6 pad 9: /OUT_B -> Net-(P6-Pad9)
- R4 pad 2: /VB1_3 -> /VB1_2
- R5 pad 2: /VB2_3 -> /VB2_2
Routing:
- net /OUT: track 43.9 -> 25.9 mm, vias 0 -> 1
- net /VB1_2: track 0.00 -> 17.6 mm
- net /VB2_2: track 0.00 -> 13.9 mm
- net /VB1_3: track 13.5 -> 0.00 mm
- net /VP_OUT: track 13.3 -> 0.00 mm
- net /VB2_3: track 12.7 -> 0.00 mm
- net /BAT-: track 10.2 -> 3.72 mm
- net /VP_1: track 7.25 -> 12.9 mm, vias 0 -> 1
- net /OUT_B: track 33.9 -> 37.8 mm
- net /OUT_N: track 44.1 -> 46.9 mm
- net Net-(C3-Pad1): track 24.7 -> 22.7 mm
- net Net-(C3-Pad2): track 26.1 -> 27.8 mm
- net /HPF_OUT: track 31.7 -> 32.4 mm
