File: BGP_V1/VOL/VOL.sch (KiCad schematic (older format))
At the start: 33 parts, among them IC1 TC7660SO-08, P1 CONN_01X03, P2 CONN_01X02, P3 CONN_01X05, P4 CONN_01X05, P5 CONN_01X05, P6 Conn_01x14, P7 CONN_02X02, U1 OPA2170

Commit message: Further component refinement in V1
Parts:
- C8: footprint Capacitors_SMD:C_0805_HandSoldering -> Capacitors_Tantalum_SMD:TantalC_SizeS_EIA-3216
Changed lines of the file:
@@
 LIBS:contrib
 LIBS:valves
-LIBS:MC_TC7660
 LIBS:VOL-cache
 EELAYER 25 0
@@
 F 0 "C8" H 7360 4370 50  0000 L CNN
 F 1 "22u" H 7360 4220 50  0000 L CNN
-F 2 "Capacitors_SMD:C_0805_HandSoldering" H 7350 4300 50  0001 C CNN
+F 2 "Capacitors_Tantalum_SMD:TantalC_SizeS_EIA-3216" H 7350 4300 50  0001 C CNN
 F 3 "" H 7350 4300 50  0000 C CNN
 	1    7350 4300

Commit message: Error found/corrected in 1_VOL. Modified to use ALPS RK097 dual shaft, quad gang.
Parts:
- removed P6: Conn_01x14, LIBS:Potentiometer_TT_P08X_Quad_Vertical_Dual_Shaft, symbol Conn_01x14
- added P6: CONN_01X12, LIBS:Potentiometer_Alps_RK097_Quad_Vertical_Dual_Shaft, symbol CONN_01X12
- added R11, R12: 11k, Resistors_SMD:R_0603_HandSoldering, symbol R_Small
- R10: value 22k -> 11k
- R9: value 18k -> 8.45k
Connections:
- net BAT-: now also P1.3 (P3); no longer P1.1 (P1)
- net Earth: now also P1.1 (P1), P6.1 (P1), P6.10 (P10), P6.4 (P4), R11.1, R12.1; no longer P1.3 (P3)
- net OUT: now also P6.11 (P11)
- net OUT_B: now also P6.3 (P3), R11.2
- net OUT_N: now also P6.6 (P6), R12.2
- net VP_1: now also P6.12 (P12)
- net VB1_3 renamed VB1_2
- net VB1_2: now also P6.2 (P2)
- net VB2_3 renamed VB2_2
- net VB2_2: now also P6.5 (P5)
Changed lines of the file:
@@
 Text Label 5500 3500 1    60   ~ 0
 VB1_1
+Text Label 5700 3500 1    60   ~ 0
+VB1_2
 Text Label 5600 3500 1    60   ~ 0
-VB1_2
-Text Label 5700 3500 1    60   ~ 0
 VB1_3
 Text Label 6500 4000 1    60   ~ 0
@@
 Text Label 5500 3950 1    60   ~ 0
 VB2_1
+Text Label 5700 3950 1    60   ~ 0
+VB2_2
 Text Label 5600 3950 1    60   ~ 0
-VB2_2
-Text Label 5700 3950 1    60   ~ 0
 VB2_3
 Text Label 5400 3500 2    60   ~ 0
@@
 Text Label 7500 4300 1    60   ~ 0
 VP_1
-Text Label 8950 4000 2    60   ~ 0
+Text Label 8900 4750 2    60   ~ 0
 VP_1
-Text Label 8950 3800 2    60   ~ 0
+Text Label 8900 4550 2    60   ~ 0
 VP_3
-Text Label 8950 3900 2    60   ~ 0
-VP_OUT
-Text Label 8950 4300 2    60   ~ 0
+Text Label 8900 4650 2    60   ~ 0
+OUT
+Text Label 8900 3850 2    60   ~ 0
 VB1_1
-Text Label 8950 4200 2    60   ~ 0
+Text Label 8900 3750 2    60   ~ 0
 VB1_2
-Text Label 8950 4100 2    60   ~ 0
+Text Label 8900 3650 2    60   ~ 0
 VB1_3
-Text Label 8950 4600 2    60   ~ 0
+Text Label 8900 4150 2    60   ~ 0
 VB2_1
-Text Label 8950 4500 2    60   ~ 0
+Text Label 8900 4050 2    60   ~ 0
 VB2_2
-Text Label 8950 4400 2    60   ~ 0
+Text Label 8900 3950 2    60   ~ 0
 VB2_3
 $Comp
@@
 L Earth #PWR011
 U 1 1 5A4E0247
-P 3600 2400
-F 0 "#PWR011" H 3600 2150 50  0001 C CNN
-F 1 "Earth" H 3600 2250 50  0001 C CNN
-F 2 "" H 3600 2400 50  0000 C CNN
-F 3 "" H 3600 2400 50  0000 C CNN
-	1    3600 2400
+P 3600 2600
+F 0 "#PWR011" H 3600 2350 50  0001 C CNN
+F 1 "Earth" H 3600 2450 50  0001 C CNN
+F 2 "" H 3600 2600 50  0000 C CNN
+F 3 "" H 3600 2600 50  0000 C CNN
+	1    3600 2600
 	0    -1   -1   0
 $EndComp
@@
 	0    1    1    0
 $EndComp
-Text Label 3600 2600 0    60   ~ 0
+Text Label 3600 2400 0    60   ~ 0
 BAT-
 $Comp
@@
 P 7650 4300
 F 0 "R9" H 7680 4320 50  0000 L CNN
-F 1 "18k" H 7680 4260 50  0000 L CNN
+F 1 "8.45k" H 7680 4260 50  0000 L CNN
 F 2 "Resistors_SMD:R_0603_HandSoldering" H 7650 4300 50  0001 C CNN
 F 3 "" H 7650 4300 50  0000 C CNN
@@
 P 7650 4600
 F 0 "R10" H 7680 4620 50  0000 L CNN
-F 1 "22k" H 7680 4560 50  0000 L CNN
+F 1 "11k" H 7680 4560 50  0000 L CNN
 F 2 "Resistors_SMD:R_0603_HandSoldering" H 7650 4600 50  0001 C CNN
 F 3 "" H 7650 4600 50  0000 C CNN
@@
 OUT
 $Comp
-L Conn_01x14 P6
-U 1 1 5A5672C2
-P 9150 4100
-F 0 "P6" H 9150 4800 50  0000 C CNN
-F 1 "Conn_01x14" H 9150 3300 50  0000 C CNN
-F 2 "LIBS:Potentiometer_TT_P08X_Quad_Vertical_Dual_Shaft" H 9150 4100 50  0001 C CNN
-F 3 "" H 9150 4100 50  0001 C CNN
-	1    9150 4100
+L CONN_01X12 P6
+U 1 1 5A5D73F9
+P 9100 4200
+F 0 "P6" H 9100 4850 50  0000 C CNN
+F 1 "CONN_01X12" V 9200 4200 50  0000 C CNN
+F 2 "LIBS:Potentiometer_Alps_RK097_Quad_Vertical_Dual_Shaft" H 9100 4200 50  0001 C CNN
+F 3 "" H 9100 4200 50  0000 C CNN
+	1    9100 4200
 	1    0    0    -1
 $EndComp
-Text Label 8950 4700 2    60   ~ 0
-VP_OUT
-Text Label 8950 4800 2    60   ~ 0
-OUT
+$Comp
+L R_Small R11
+U 1 1 5A5D792F
+P 7650 3500
+F 0 "R11" H 7680 3520 50  0000 L CNN
+F 1 "11k" H 7680 3460 50  0000 L CNN
+F 2 "Resistors_SMD:R_0603_HandSoldering" H 7650 3500 50  0001 C CNN
+F 3 "" H 7650 3500 50  0000 C CNN
+	1    7650 3500
+	0    1    1    0
+$EndComp
+$Comp
+L R_Small R12
+U 1 1 5A5D7B92
+P 7650 3800
+F 0 "R12" H 7680 3820 50  0000 L CNN
+F 1 "11k" H 7680 3760 50  0000 L CNN
+F 2 "Resistors_SMD:R_0603_HandSoldering" H 7650 3800 50  0001 C CNN
+F 3 "" H 7650 3800 50  0000 C CNN
+	1    7650 3800
+	0    1    1    0
+$EndComp
+Text Label 7550 3500 2    60   ~ 0
+VB1_1
+Text Label 7750 3500 0    60   ~ 0
+VB1_3
+Text Label 7550 3800 2    60   ~ 0
+VB2_1
+Text Label 7750 3800 0    60   ~ 0
+VB2_3
 $EndSCHEMATC
