File: BGP_F0/BT_STACK/BT_STACK.kicad_pcb (KiCad board)
At the start: 2 copper layers, 24 x 26 mm, 18 parts, among them P1 CONN_01X05, P2 CONN_01X02, P3 CONN_01X04, U1 MC33178

Commit message: Some Changes
Parts:
- moved RV1 0.10 mm to (148.2, 72.8)
Changed lines of the file:
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@@
     (links 34)
     (no_connects 0)
-    (area 139.924999 68.924999 164.075001 95.075001)
+    (area 139.924999 68.164286 164.075001 95.955)
     (thickness 1.6)
     (drawings 8)
@@
     )
   )
-  (module LIBS:Potentiometer_Alpha_Double_Vertical_Dual_Shaft (layer B.Cu)
-    (at 148.35 72.8 90)
-    (descr "Potentiometer, vertically mounted, Omeg PC16PU, Omeg PC16PU, Omeg PC16PU, Vishay/Spectrol 248GJ/249GJ Single, Vishay/Spectrol 248GJ/249GJ Single, Vishay/Spectrol 248GJ/249GJ Single, Vishay/Spectrol 248GH/249GH Single, Vishay/Spectrol 148/149 Single, Vishay/Spectrol 148/149 Single, Vishay/Spectrol 148/149 Single, Vishay/Spectrol 148A/149A Single with mounting plates, Vishay/Spectrol 148/149 Double, Vishay/Spectrol 148A/149A Double with mounting plates, Piher PC-16 Single, Piher PC-16 Single, Piher PC-16 Single, Piher PC-16SV Single, Piher PC-16 Double, Piher PC-16 Triple, Piher T16H Single, Piher T16L Single, Piher T16H Double, Alps RK163 Single, Alps RK163 Double, Alps RK097 Single, Alps RK097 Double, http://www.alps.com/prod/info/E/HTML/Potentiometer/RotaryPotentiometers/RK097/RK09712100AV.html")
-    (tags "Potentiometer vertical  Omeg PC16PU  Omeg PC16PU  Omeg PC16PU  Vishay/Spectrol 248GJ/249GJ Single  Vishay/Spectrol 248GJ/249GJ Single  Vishay/Spectrol 248GJ/249GJ Single  Vishay/Spectrol 248GH/249GH Single  Vishay/Spectrol 148/149 Single  Vishay/Spectrol 148/149 Single  Vishay/Spectrol 148/149 Single  Vishay/Spectrol 148A/149A Single with mounting plates  Vishay/Spectrol 148/149 Double  Vishay/Spectrol 148A/149A Double with mounting plates  Piher PC-16 Single  Piher PC-16 Single  Piher PC-16 Single  Piher PC-16SV Single  Piher PC-16 Double  Piher PC-16 Triple  Piher T16H Single  Piher T16L Single  Piher T16H Double  Alps RK163 Single  Alps RK163 Double  Alps RK097 Single  Alps RK097 Double Dual Shaft")
-    (fp_text reference RV1 (at 1 11.05 90) (layer B.SilkS)
-      (effects (font (size 0.6 0.6) (thickness 0.15)) (justify mirror))
-    )
-    (fp_text value DUAL_POT (at 2.15 -4 90) (layer B.Fab) hide
-      (effects (font (size 0.6 0.6) (thickness 0.15)) (justify mirror))
-    )
-    (fp_line (start -11.7 10.35) (end -11.7 -2.85) (layer B.Fab) (width 0.1))
-    (fp_line (start -11.7 -2.85) (end 1.8 -2.85) (layer B.Fab) (width 0.1))
-    (fp_line (start 1.8 -2.85) (end 1.8 10.35) (layer B.Fab) (width 0.1))
-    (fp_line (start 1.8 10.35) (end -11.7 10.35) (layer B.Fab) (width 0.1))
-    (fp_line (start -11.76 10.4) (end 1.86 10.4) (layer B.SilkS) (width 0.12))
-    (fp_line (start -11.76 -2.91) (end 1.86 -2.91) (layer B.SilkS) (width 0.12))
-    (fp_line (start -11.76 10.4) (end -11.76 -2.91) (layer B.SilkS) (width 0.12))
-    (fp_line (start 1.86 10.4) (end 1.86 -2.91) (layer B.SilkS) (width 0.12))
-    (fp_line (start -12.15 10.6) (end -12.15 -3.1) (layer B.CrtYd) (width 0.05))
-    (fp_line (start -12.15 -3.1) (end 2.1 -3.1) (layer B.CrtYd) (width 0.05))
-    (fp_line (start 2.1 -3.1) (end 2.1 10.6) (layer B.CrtYd) (width 0.05))
-    (fp_line (start 2.1 10.6) (end -12.15 10.6) (layer B.CrtYd) (width 0.05))
-    (pad 3 thru_hole circle (at 0 7.3 90) (size 1.8 1.8) (drill 1) (layers *.Cu *.Mask)
-      (net 8 /B+))
-    (pad 2 thru_hole circle (at 0 3.65 90) (size 1.8 1.8) (drill 1) (layers *.Cu *.Mask)
-      (net 13 /BW))
-    (pad 1 thru_hole circle (at 0 0 90) (size 1.8 1.8) (drill 1) (layers *.Cu *.Mask)
-      (net 9 /B-))
-    (pad 6 thru_hole circle (at -5 7.3 90) (size 1.8 1.8) (drill 1) (layers *.Cu *.Mask)
-      (net 15 /T+))
-    (pad 5 thru_hole circle (at -5 3.65 90) (size 1.8 1.8) (drill 1) (layers *.Cu *.Mask)
-      (net 5 /TW))
-    (pad 4 thru_hole circle (at -5 0 90) (size 1.8 1.8) (drill 1) (layers *.Cu *.Mask)
-      (net 14 /T-))
-    (model Potentiometers.3dshapes/Potentiometer_Alps_RK097_Double_Vertical.wrl
-      (at (xyz 0 0 0))
-      (scale (xyz 0.393701 0.393701 0.393701))
-      (rotate (xyz 0 0 0))
-    )
-  )
   (module Connectors_JST:JST_PH_B5B-PH-K_05x2.00mm_Straight (layer F.Cu)
     (at 142.7 91.3)
@@
     )
   )
+  (module LIBS:Potentiometer_Alpha_Double_Vertical_Dual_Shaft (layer B.Cu)
+    (at 148.25 72.8 90)
+    (descr "Potentiometer, vertically mounted, Omeg PC16PU, Omeg PC16PU, Omeg PC16PU, Vishay/Spectrol 248GJ/249GJ Single, Vishay/Spectrol 248GJ/249GJ Single, Vishay/Spectrol 248GJ/249GJ Single, Vishay/Spectrol 248GH/249GH Single, Vishay/Spectrol 148/149 Single, Vishay/Spectrol 148/149 Single, Vishay/Spectrol 148/149 Single, Vishay/Spectrol 148A/149A Single with mounting plates, Vishay/Spectrol 148/149 Double, Vishay/Spectrol 148A/149A Double with mounting plates, Piher PC-16 Single, Piher PC-16 Single, Piher PC-16 Single, Piher PC-16SV Single, Piher PC-16 Double, Piher PC-16 Triple, Piher T16H Single, Piher T16L Single, Piher T16H Double, Alps RK163 Single, Alps RK163 Double, Alps RK097 Single, Alps RK097 Double, http://www.alps.com/prod/info/E/HTML/Potentiometer/RotaryPotentiometers/RK097/RK09712100AV.html")
+    (tags "Potentiometer vertical  Omeg PC16PU  Omeg PC16PU  Omeg PC16PU  Vishay/Spectrol 248GJ/249GJ Single  Vishay/Spectrol 248GJ/249GJ Single  Vishay/Spectrol 248GJ/249GJ Single  Vishay/Spectrol 248GH/249GH Single  Vishay/Spectrol 148/149 Single  Vishay/Spectrol 148/149 Single  Vishay/Spectrol 148/149 Single  Vishay/Spectrol 148A/149A Single with mounting plates  Vishay/Spectrol 148/149 Double  Vishay/Spectrol 148A/149A Double with mounting plates  Piher PC-16 Single  Piher PC-16 Single  Piher PC-16 Single  Piher PC-16SV Single  Piher PC-16 Double  Piher PC-16 Triple  Piher T16H Single  Piher T16L Single  Piher T16H Double  Alps RK163 Single  Alps RK163 Double  Alps RK097 Single  Alps RK097 Double Dual Shaft")
+    (fp_text reference RV1 (at 2.7 9.75 180) (layer B.SilkS)
+      (effects (font (size 0.6 0.6) (thickness 0.15)) (justify mirror))
+    )
+    (fp_text value DUAL_POT (at 2.15 -3.9 90) (layer B.Fab) hide
+      (effects (font (size 0.6 0.6) (thickness 0.15)) (justify mirror))
+    )
+    (fp_line (start -11.7 10.45) (end -11.7 -2.75) (layer B.Fab) (width 0.1))
+    (fp_line (start -11.7 -2.75) (end 1.8 -2.75) (layer B.Fab) (width 0.1))
+    (fp_line (start 1.8 -2.75) (end 1.8 10.45) (layer B.Fab) (width 0.1))
+    (fp_line (start 1.8 10.45) (end -11.7 10.45) (layer B.Fab) (width 0.1))
+    (fp_line (start -11.76 10.5) (end 1.86 10.5) (layer B.SilkS) (width 0.12))
+    (fp_line (start -11.76 -2.81) (end 1.86 -2.81) (layer B.SilkS) (width 0.12))
+    (fp_line (start -11.76 10.5) (end -11.76 -2.81) (layer B.SilkS) (width 0.12))
+    (fp_line (start 1.86 10.5) (end 1.86 -2.81) (layer B.SilkS) (width 0.12))
+    (fp_line (start -12.15 10.7) (end -12.15 -3) (layer B.CrtYd) (width 0.05))
+    (fp_line (start -12.15 -3) (end 2.1 -3) (layer B.CrtYd) (width 0.05))
+    (fp_line (start 2.1 -3) (end 2.1 10.7) (layer B.CrtYd) (width 0.05))
+    (fp_line (start 2.1 10.7) (end -12.15 10.7) (layer B.CrtYd) (width 0.05))
+    (pad 3 thru_hole circle (at 0 7.5 90) (size 1.8 1.8) (drill 1) (layers *.Cu *.Mask)
+      (net 8 /B+))
+    (pad 2 thru_hole circle (at 0 3.75 90) (size 1.8 1.8) (drill 1) (layers *.Cu *.Mask)
+      (net 13 /BW))
+    (pad 1 thru_hole circle (at 0 0 90) (size 1.8 1.8) (drill 1) (layers *.Cu *.Mask)
+      (net 9 /B-))
+    (pad 6 thru_hole circle (at -5 7.5 90) (size 1.8 1.8) (drill 1) (layers *.Cu *.Mask)
+      (net 15 /T+))
+    (pad 5 thru_hole circle (at -5 3.75 90) (size 1.8 1.8) (drill 1) (layers *.Cu *.Mask)
+      (net 5 /TW))
+    (pad 4 thru_hole circle (at -5 0 90) (size 1.8 1.8) (drill 1) (layers *.Cu *.Mask)
+      (net 14 /T-))
+    (model Potentiometers.3dshapes/Potentiometer_Alps_RK097_Double_Vertical.wrl
+      (at (xyz 0 0 0))
+      (scale (xyz 0.393701 0.393701 0.393701))
+      (rotate (xyz 0 0 0))
+    )
+  )

Commit message: F0 Final
Parts:
- C4: footprint Capacitors_SMD:C_0805_HandSoldering -> Capacitors_SMD:C_0603
Routing:
- net Net-(C3-Pad2): track 16.8 -> 17.3 mm
Changed lines of the file:
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@@
     (links 34)
     (no_connects 0)
-    (area 139.924999 68.164286 164.075001 95.955)
+    (area 139.924999 68.924999 164.075001 95.075001)
     (thickness 1.6)
     (drawings 8)
@@
   )
   (module Capacitors_SMD:C_0805_HandSoldering (layer F.Cu)
-    (at 152 81.6)
-    (descr "Capacitor SMD 0805, hand soldering")
-    (tags "capacitor 0805")
-    (attr smd)
-    (fp_text reference C4 (at -1.8 -1.4) (layer F.SilkS)
-      (effects (font (size 0.6 0.6) (thickness 0.15)))
-    )
-    (fp_text value 470p (at 0 2.1) (layer F.Fab) hide
-      (effects (font (size 0.6 0.6) (thickness 0.15)))
-    )
-    (fp_line (start -2.3 -1) (end 2.3 -1) (layer F.CrtYd) (width 0.05))
-    (fp_line (start -2.3 1) (end 2.3 1) (layer F.CrtYd) (width 0.05))
-    (fp_line (start -2.3 -1) (end -2.3 1) (layer F.CrtYd) (width 0.05))
-    (fp_line (start 2.3 -1) (end 2.3 1) (layer F.CrtYd) (width 0.05))
-    (fp_line (start 0.5 -0.85) (end -0.5 -0.85) (layer F.SilkS) (width 0.15))
-    (fp_line (start -0.5 0.85) (end 0.5 0.85) (layer F.SilkS) (width 0.15))
-    (pad 1 smd rect (at -1.25 0) (size 1.5 1.25) (layers F.Cu F.Paste F.Mask)
-      (net 7 /MID_I))
-    (pad 2 smd rect (at 1.25 0) (size 1.5 1.25) (layers F.Cu F.Paste F.Mask)
-      (net 6 "Net-(C3-Pad2)"))
-    (model Capacitors_SMD.3dshapes/C_0805_HandSoldering.wrl
-      (at (xyz 0 0 0))
-      (scale (xyz 1 1 1))
-      (rotate (xyz 0 0 0))
-    )
-  )
-  (module Capacitors_SMD:C_0805_HandSoldering (layer F.Cu)
     (at 152 75.4)
     (descr "Capacitor SMD 0805, hand soldering")
@@
       (at (xyz 0 0 0))
       (scale (xyz 0.393701 0.393701 0.393701))
+      (rotate (xyz 0 0 0))
+    )
+  )
+  (module Capacitors_SMD:C_0603 (layer F.Cu)
+    (at 152 81.6)
+    (descr "Capacitor SMD 0603, reflow soldering, AVX (see smccp.pdf)")
+    (tags "capacitor 0603")
+    (attr smd)
+    (fp_text reference C4 (at -0.9 -1.075001) (layer F.SilkS)
+      (effects (font (size 0.6 0.6) (thickness 0.15)))
+    )
+    (fp_text value 470p (at 0 1.9) (layer F.Fab) hide
+      (effects (font (size 0.6 0.6) (thickness 0.15)))
+    )
+    (fp_line (start -1.45 -0.75) (end 1.45 -0.75) (layer F.CrtYd) (width 0.05))
+    (fp_line (start -1.45 0.75) (end 1.45 0.75) (layer F.CrtYd) (width 0.05))
+    (fp_line (start -1.45 -0.75) (end -1.45 0.75) (layer F.CrtYd) (width 0.05))
+    (fp_line (start 1.45 -0.75) (end 1.45 0.75) (layer F.CrtYd) (width 0.05))
+    (fp_line (start -0.35 -0.6) (end 0.35 -0.6) (layer F.SilkS) (width 0.15))
+    (fp_line (start 0.35 0.6) (end -0.35 0.6) (layer F.SilkS) (width 0.15))
+    (pad 1 smd rect (at -0.75 0) (size 0.8 0.75) (layers F.Cu F.Paste F.Mask)
+      (net 7 /MID_I))
+    (pad 2 smd rect (at 0.75 0) (size 0.8 0.75) (layers F.Cu F.Paste F.Mask)
+      (net 6 "Net-(C3-Pad2)"))
+    (model Capacitors_SMD.3dshapes/C_0603.wrl
+      (at (xyz 0 0 0))
+      (scale (xyz 1 1 1))
       (rotate (xyz 0 0 0))
     )
@@
   (segment (start 159.15 82.65) (end 159.1 82.6) (width 0.3) (layer F.Cu) (net 5))
   (via (at 159.1 82.6) (size 0.6) (drill 0.4) (layers F.Cu B.Cu) (net 5))
+  (segment (start 155.8 81.6) (end 152.75 81.6) (width 0.3) (layer F.Cu) (net 6))
   (segment (start 156.9 82.7) (end 155.8 81.6) (width 0.3) (layer F.Cu) (net 6))
-  (segment (start 155.8 81.6) (end 153.25 81.6) (width 0.3) (layer F.Cu) (net 6))
   (segment (start 156.9 82.75) (end 156.9 82.7) (width 0.3) (layer F.Cu) (net 6))
   (segment (start 156.9 85.8) (end 156.065 86.635) (width 0.3) (layer F.Cu) (net 6))
@@
   (segment (start 161.525 83.8) (end 159 81.275) (width 0.3) (layer F.Cu) (net 6))
   (segment (start 159 81.275) (end 159 80.8) (width 0.3) (layer F.Cu) (net 6))
+  (segment (start 151.25 81.6) (end 151.25 82.275) (width 0.3) (layer F.Cu) (net 7))
+  (segment (start 151.25 82.275) (end 151.8 82.825) (width 0.3) (layer F.Cu) (net 7))
+  (segment (start 151.8 82.825) (end 151.8 85.48) (width 0.3) (layer F.Cu) (net 7))
+  (segment (start 151.25 81.6) (end 148.5 81.6) (width 0.3) (layer F.Cu) (net 7))
   (segment (start 154.225 87.905) (end 154.7 87.905) (width 0.3) (layer F.Cu) (net 7))
   (segment (start 151.8 85.48) (end 154.225 87.905) (width 0.3) (layer F.Cu) (net 7))
-  (segment (start 151.8 82.525) (end 151.8 85.48) (width 0.3) (layer F.Cu) (net 7))
-  (segment (start 150.875 81.6) (end 151.8 82.525) (width 0.3) (layer F.Cu) (net 7))
-  (segment (start 150.75 81.6) (end 150.875 81.6) (width 0.3) (layer F.Cu) (net 7))
   (segment (start 145 79) (end 145 78.4) (width 0.3) (layer F.Cu) (net 7))
   (segment (start 145 78.4) (end 142.8 76.2) (width 0.3) (layer F.Cu) (net 7))
@@
   (segment (start 145 79) (end 145.9 79) (width 0.3) (layer F.Cu) (net 7))
   (segment (start 145.9 79) (end 148.5 81.6) (width 0.3) (layer F.Cu) (net 7))
-  (segment (start 148.5 81.6) (end 150.75 81.6) (width 0.3) (layer F.Cu) (net 7))
   (segment (start 154.7 87.905) (end 154.7 88.505) (width 0.3) (layer F.Cu) (net 7))
   (segment (start 154.7 88.505) (end 155.3 89.105) (width 0.3) (layer F.Cu) (net 7))

Commit message: Various - BOM complete
Parts:
- added C6: 470p, Capacitors_SMD:C_0603, F.Cu at (143.4, 86.5)
- R2, R4: value 4.7k -> 4.99k
- R6, R7: value 22k -> 20k
Routing:
- net Net-(C6-Pad2): track 10.4 -> 19.9 mm
- net Net-(C6-Pad1): track 8.83 -> 12.6 mm
Changed lines of the file:
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@@
-(kicad_pcb (version 4) (host pcbnew 4.0.4-1.fc24-product)
+(kicad_pcb (version 4) (host pcbnew 4.0.7)
   (general
-    (links 34)
+    (links 36)
     (no_connects 0)
     (area 139.924999 68.924999 164.075001 95.075001)
     (thickness 1.6)
     (drawings 8)
-    (tracks 123)
+    (tracks 131)
     (zones 0)
-    (modules 18)
+    (modules 19)
     (nets 18)
   )
@@
   (net 14 /T-)
   (net 15 /T+)
-  (net 16 "Net-(R6-Pad1)")
-  (net 17 "Net-(R7-Pad1)")
+  (net 16 "Net-(C6-Pad2)")
+  (net 17 "Net-(C6-Pad1)")
   (net_class Default "This is the default net class."
     (clearance 0.3)
@@
     (add_net Earth)
     (add_net "Net-(C3-Pad2)")
-    (add_net "Net-(R6-Pad1)")
-    (add_net "Net-(R7-Pad1)")
+    (add_net "Net-(C6-Pad1)")
+    (add_net "Net-(C6-Pad2)")
   )
   (net_class PWR ""
@@
       (net 12 /MID_R))
     (pad 6 smd rect (at 2.7 0.635 180) (size 1.55 0.6) (layers F.Cu F.Paste F.Mask)
-      (net 16 "Net-(R6-Pad1)"))
+      (net 16 "Net-(C6-Pad2)"))
     (pad 7 smd rect (at 2.7 -0.635 180) (size 1.55 0.6) (layers F.Cu F.Paste F.Mask)
-      (net 17 "Net-(R7-Pad1)"))
+      (net 17 "Net-(C6-Pad1)"))
     (pad 8 smd rect (at 2.7 -1.905 180) (size 1.55 0.6) (layers F.Cu F.Paste F.Mask)
       (net 1 /V+))
@@
       (net 3 /MID_O))
     (pad 2 smd rect (at 1.1 0) (size 1.2 0.9) (layers F.Cu F.Paste F.Mask)
-      (net 17 "Net-(R7-Pad1)"))
+      (net 17 "Net-(C6-Pad1)"))
     (model Resistors_SMD.3dshapes/R_0603_HandSoldering.wrl
       (at (xyz 0 0 0))
@@
       (effects (font (size 0.6 0.6) (thickness 0.15)))
     )
-    (fp_text value 4.7k (at 0 1.9) (layer F.Fab) hide
+    (fp_text value 4.99k (at 0 1.9) (layer F.Fab) hide
       (effects (font (size 0.6 0.6) (thickness 0.15)))
     )
@@
       (effects (font (size 0.6 0.6) (thickness 0.15)))
     )
-    (fp_text value 22k (at 0 1.9) (layer F.Fab) hide
+    (fp_text value 20k (at 0 1.9) (layer F.Fab) hide
       (effects (font (size 0.6 0.6) (thickness 0.15)))
     )
@@
     (fp_line (start -0.5 -0.675) (end 0.5 -0.675) (layer F.SilkS) (width 0.15))
     (pad 1 smd rect (at -1.1 0) (size 1.2 0.9) (layers F.Cu F.Paste F.Mask)
-      (net 17 "Net-(R7-Pad1)"))
+      (net 17 "Net-(C6-Pad1)"))
     (pad 2 smd rect (at 1.1 0) (size 1.2 0.9) (layers F.Cu F.Paste F.Mask)
-      (net 16 "Net-(R6-Pad1)"))
+      (net 16 "Net-(C6-Pad2)"))
     (model Resistors_SMD.3dshapes/R_0603_HandSoldering.wrl
       (at (xyz 0 0 0))
@@
       (effects (font (size 0.6 0.6) (thickness 0.15)))
     )
-    (fp_text value 4.7k (at 0 1.9) (layer F.Fab) hide
+    (fp_text value 4.99k (at 0 1.9) (layer F.Fab) hide
       (effects (font (size 0.6 0.6) (thickness 0.15)))
     )
@@
       (effects (font (size 0.6 0.6) (thickness 0.15)))
     )
-    (fp_text value 22k (at 0 1.9) (layer F.Fab) hide
+    (fp_text value 20k (at 0 1.9) (layer F.Fab) hide
       (effects (font (size 0.6 0.6) (thickness 0.15)))
     )
@@
     (fp_line (start -0.5 -0.675) (end 0.5 -0.675) (layer F.SilkS) (width 0.15))
     (pad 1 smd rect (at -1.1 0) (size 1.2 0.9) (layers F.Cu F.Paste F.Mask)
-      (net 16 "Net-(R6-Pad1)"))
+      (net 16 "Net-(C6-Pad2)"))
     (pad 2 smd rect (at 1.1 0) (size 1.2 0.9) (layers F.Cu F.Paste F.Mask)
       (net 7 /MID_I))
@@
     (pad 2 smd rect (at 0.75 0) (size 0.8 0.75) (layers F.Cu F.Paste F.Mask)
       (net 6 "Net-(C3-Pad2)"))
+    (model Capacitors_SMD.3dshapes/C_0603.wrl
+      (at (xyz 0 0 0))
+      (scale (xyz 1 1 1))
+      (rotate (xyz 0 0 0))
+    )
+  )
+  (module Capacitors_SMD:C_0603 (layer F.Cu)
+    (at 143.4 86.5 180)
+    (descr "Capacitor SMD 0603, reflow soldering, AVX (see smccp.pdf)")
+    (tags "capacitor 0603")
+    (attr smd)
+    (fp_text reference C6 (at -0.9 -1 360) (layer F.SilkS)
+      (effects (font (size 0.6 0.6) (thickness 0.15)))
+    )
+    (fp_text value 470p (at 0 1.5 180) (layer F.Fab) hide
+      (effects (font (size 0.6 0.6) (thickness 0.15)))
+    )
+    (fp_line (start 1.4 0.65) (end -1.4 0.65) (layer F.CrtYd) (width 0.05))
+    (fp_line (start 1.4 0.65) (end 1.4 -0.65) (layer F.CrtYd) (width 0.05))
+    (fp_line (start -1.4 -0.65) (end -1.4 0.65) (layer F.CrtYd) (width 0.05))
+    (fp_line (start -1.4 -0.65) (end 1.4 -0.65) (layer F.CrtYd) (width 0.05))
+    (fp_line (start 0.35 0.6) (end -0.35 0.6) (layer F.SilkS) (width 0.12))
+    (fp_line (start -0.35 -0.6) (end 0.35 -0.6) (layer F.SilkS) (width 0.12))
+    (fp_line (start -0.8 -0.4) (end 0.8 -0.4) (layer F.Fab) (width 0.1))
+    (fp_line (start 0.8 -0.4) (end 0.8 0.4) (layer F.Fab) (width 0.1))
+    (fp_line (start 0.8 0.4) (end -0.8 0.4) (layer F.Fab) (width 0.1))
+    (fp_line (start -0.8 0.4) (end -0.8 -0.4) (layer F.Fab) (width 0.1))
+    (fp_text user %R (at 0 0 360) (layer F.Fab) hide
+      (effects (font (size 0.3 0.3) (thickness 0.075)))
+    )
+    (pad 2 smd rect (at 0.75 0 180) (size 0.8 0.75) (layers F.Cu F.Paste F.Mask)
+      (net 16 "Net-(C6-Pad2)"))
+    (pad 1 smd rect (at -0.75 0 180) (size 0.8 0.75) (layers F.Cu F.Paste F.Mask)
+      (net 17 "Net-(C6-Pad1)"))
     (model Capacitors_SMD.3dshapes/C_0603.wrl
       (at (xyz 0 0 0))
@@
   (segment (start 146.55 76) (end 148.35 77.8) (width 0.3) (layer F.Cu) (net 14))
   (segment (start 159 77.8) (end 155.65 77.8) (width 0.3) (layer F.Cu) (net 15))
+  (segment (start 142.65 86.5) (end 141.95 86.5) (width 0.3) (layer F.Cu) (net 16))
+  (segment (start 141.95 86.5) (end 141.4 85.95) (width 0.3) (layer F.Cu) (net 16))
+  (segment (start 141.4 85.95) (end 141.4 79.6) (width 0.3) (layer F.Cu) (net 16))
+  (segment (start 141.4 79.6) (end 142 79) (width 0.3) (layer F.Cu) (net 16))
+  (segment (start 142 79) (end 142.8 79) (width 0.3) (layer F.Cu) (net 16))
   (segment (start 145 81.5) (end 145.9 81.5) (width 0.3) (layer F.Cu) (net 16))
   (segment (start 145.9 81.5) (end 146.7 82.3) (width 0.3) (layer F.Cu) (net 16))
@@
   (segment (start 142.95 79) (end 145 81.05) (width 0.3) (layer F.Cu) (net 16))
   (segment (start 145 81.05) (end 145 81.5) (width 0.3) (layer F.Cu) (net 16))
+  (segment (start 145.1 86.5) (end 145.235 86.635) (width 0.3) (layer F.Cu) (net 17))
+  (segment (start 145.235 86.635) (end 147.885 86.635) (width 0.3) (layer F.Cu) (net 17))
+  (segment (start 144.15 86.5) (end 145.1 86.5) (width 0.3) (layer F.Cu) (net 17))
   (segment (start 149.3 86.635) (end 147.885 86.635) (width 0.3) (layer F.Cu) (net 17))
   (segment (start 147.885 86.635) (end 145.25 84) (width 0.3) (layer F.Cu) (net 17))
