File: BGP_F0/BT_STACK/BT_STACK.sch (KiCad schematic (older format))
At the start: 19 parts, among them P1 CONN_01X05, P3 CONN_01X04, U1 MC33178

Commit message: F0 BT stack changed slightly
Parts:
- R2, R4: value 4.99k -> 6.8k
Connections:
- net Earth: now also P1.5 (P5); no longer P1.1 (P1)
- net IN: now also P1.1 (P1); no longer P1.5 (P5)
- net MID_I: now also P3.4 (P4); no longer P3.1 (P1)
- net MID_O: now also P3.2 (P2); no longer P3.3 (P3)
- net MID_R: now also P3.3 (P3); no longer P3.2 (P2)
- net OUT: now also P1.2 (P2); no longer P1.4 (P4)
- net Vref: now also P1.4 (P4), P3.1 (P1); no longer P1.2 (P2), P3.4 (P4)
Changed lines of the file:
@@
 P 4950 3750
 F 0 "R2" H 4980 3770 50  0000 L CNN
-F 1 "4.99k" H 4980 3710 50  0000 L CNN
+F 1 "6.8k" H 4980 3710 50  0000 L CNN
 F 2 "Resistors_SMD:R_0603_HandSoldering" H 4950 3750 50  0001 C CNN
 F 3 "" H 4950 3750 50  0000 C CNN
@@
 P 5850 3750
 F 0 "R4" H 5880 3770 50  0000 L CNN
-F 1 "4.99k" H 5880 3710 50  0000 L CNN
+F 1 "6.8k" H 5880 3710 50  0000 L CNN
 F 2 "Resistors_SMD:R_0603_HandSoldering" H 5850 3750 50  0001 C CNN
 F 3 "" H 5850 3750 50  0000 C CNN
@@
 F 3 "" H 3750 2500 50  0000 C CNN
 	1    3750 2500
-	-1   0    0    1
+	-1   0    0    -1
 $EndComp
 $Comp
@@
 F 3 "" H 8800 2450 50  0000 C CNN
 	1    8800 2450
-	1    0    0    1
+	1    0    0    -1
 $EndComp
 Text Label 8600 2300 2    60   ~ 0

Commit message: F0 Conn changes
Connections:
- net Earth: now also P1.1 (P1); no longer P1.5 (P5)
- net IN: now also P1.5 (P5); no longer P1.1 (P1)
- net OUT: now also P1.4 (P4); no longer P1.2 (P2)
- net Vref: now also P1.2 (P2); no longer P1.4 (P4)
Changed lines of the file:
@@
 F 3 "" H 3750 2500 50  0000 C CNN
 	1    3750 2500
-	-1   0    0    -1
+	-1   0    0    1
 $EndComp
 $Comp
