File: FET_TS/TST.kicad_pcb (KiCad board)
At the start: 2 copper layers, 30 x 28.1 mm, 5 parts, among them P1 CONN_01X02, P2 CONN_01X02, Q1 Q_NJFET_DSG

Commit message: Mods and gerbers done
Parts:
- moved R1 0.45 mm to (184.6, 73.1)
- moved P2 0.45 mm to (202.7, 89.4)
- moved Q1 0.45 mm to (184.6, 81.9)
- moved R2 0.45 mm to (184.6, 90.9)
- moved P1 0.45 mm to (202.8, 75.5)
Other:
- board size 30 x 28.1 mm -> 30 x 26 mm
Changed lines of the file:
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@@
   (general
     (links 7)
-    (no_connects 2)
-    (area 176.324999 68.124999 206.475001 96.375001)
+    (no_connects 0)
+    (area 175.924999 69.924999 207.933334 95.075001)
     (thickness 1.6)
     (drawings 8)
@@
     (visible_elements FFFFFF7F)
     (pcbplotparams
-      (layerselection 0x00030_80000001)
-      (usegerberextensions false)
+      (layerselection 0x010fc_80000001)
+      (usegerberextensions true)
       (excludeedgelayer true)
       (linewidth 0.100000)
@@
       (outputformat 1)
       (mirror false)
-      (drillshape 1)
+      (drillshape 0)
       (scaleselection 1)
-      (outputdirectory ""))
+      (outputdirectory ../GERBER/TST/))
   )
   (net 0 "")
@@
   )
   (module Pin_Headers:Pin_Header_Straight_1x02 (layer F.Cu)
-    (at 203.2 75.7 180)
+    (at 202.8 75.5 180)
     (descr "Through hole pin header")
     (tags "pin header")
@@
   )
   (module Pin_Headers:Pin_Header_Straight_1x02 (layer F.Cu)
-    (at 203.1 89.6)
+    (at 202.7 89.4)
     (descr "Through hole pin header")
     (tags "pin header")
@@
   )
   (module TO_SOT_Packages_SMD:SOT-23_Handsoldering (layer F.Cu)
-    (at 185 82.1)
+    (at 184.6 81.9)
     (descr "SOT-23, Handsoldering")
     (tags SOT-23)
@@
   )
   (module Resistors_SMD:R_0603_HandSoldering (layer F.Cu)
-    (at 185 73.3 180)
+    (at 184.6 73.1 180)
     (descr "Resistor SMD 0603, hand soldering")
     (tags "resistor 0603")
@@
   )
   (module Resistors_SMD:R_0603_HandSoldering (layer F.Cu)
-    (at 185 91.1)
+    (at 184.6 90.9)
     (descr "Resistor SMD 0603, hand soldering")
     (tags "resistor 0603")
@@
     )
   )
-  (gr_line (start 206.1 95.9) (end 206.1 68.5) (angle 90) (layer Margin) (width 0.2))
-  (gr_line (start 176.7 95.9) (end 206.1 95.9) (angle 90) (layer Margin) (width 0.2))
-  (gr_line (start 176.7 68.5) (end 176.7 95.9) (angle 90) (layer Margin) (width 0.2))
-  (gr_line (start 206.1 68.5) (end 176.7 68.5) (angle 90) (layer Margin) (width 0.2))
-  (gr_line (start 206.4 96.3) (end 206.4 68.2) (angle 90) (layer Edge.Cuts) (width 0.15))
-  (gr_line (start 176.4 96.3) (end 206.4 96.3) (angle 90) (layer Edge.Cuts) (width 0.15))
-  (gr_line (start 176.4 68.2) (end 176.4 96.3) (angle 90) (layer Edge.Cuts) (width 0.15))
-  (gr_line (start 206.4 68.2) (end 176.4 68.2) (angle 90) (layer Edge.Cuts) (width 0.15))
-  (segment (start 203.2 73.16) (end 186.24 73.16) (width 0.6) (layer F.Cu) (net 2))
-  (segment (start 186.24 73.16) (end 186.1 73.3) (width 0.6) (layer F.Cu) (net 2))
-  (segment (start 203.16 73.2) (end 203.2 73.16) (width 0.6) (layer F.Cu) (net 2))
-  (segment (start 185 93.9) (end 183.9 92.8) (width 0.6) (layer F.Cu) (net 3))
-  (segment (start 183.9 92.8) (end 183.9 91.1) (width 0.6) (layer F.Cu) (net 3))
-  (segment (start 201.34 93.9) (end 185 93.9) (width 0.6) (layer F.Cu) (net 3))
-  (segment (start 203.1 92.14) (end 201.34 93.9) (width 0.6) (layer F.Cu) (net 3))
-  (segment (start 183.9 91.1) (end 183.9 83.45) (width 0.6) (layer F.Cu) (net 3))
-  (segment (start 183.9 83.45) (end 183.5 83.05) (width 0.6) (layer F.Cu) (net 3))
-  (segment (start 183.9 73.3) (end 183.9 80.75) (width 0.6) (layer F.Cu) (net 4))
-  (segment (start 183.9 80.75) (end 183.5 81.15) (width 0.6) (layer F.Cu) (net 4))
+  (gr_line (start 205.7 95.7) (end 205.7 70.3) (angle 90) (layer Margin) (width 0.2))
+  (gr_line (start 176.3 95.7) (end 205.7 95.7) (angle 90) (layer Margin) (width 0.2))
+  (gr_line (start 176.3 70.3) (end 176.3 95.7) (angle 90) (layer Margin) (width 0.2))
+  (gr_line (start 205.7 70.3) (end 176.3 70.3) (angle 90) (layer Margin) (width 0.2))
+  (gr_line (start 206 96) (end 206 70) (angle 90) (layer Edge.Cuts) (width 0.15))
+  (gr_line (start 176 96) (end 206 96) (angle 90) (layer Edge.Cuts) (width 0.15))
+  (gr_line (start 176 70) (end 176 96) (angle 90) (layer Edge.Cuts) (width 0.15))
+  (gr_line (start 206 70) (end 176 70) (angle 90) (layer Edge.Cuts) (width 0.15))
+  (segment (start 202.8 72.96) (end 185.84 72.96) (width 0.6) (layer F.Cu) (net 2))
+  (segment (start 185.84 72.96) (end 185.7 73.1) (width 0.6) (layer F.Cu) (net 2))
+  (segment (start 202.76 73) (end 202.8 72.96) (width 0.6) (layer F.Cu) (net 2))
+  (segment (start 184.6 93.7) (end 183.5 92.6) (width 0.6) (layer F.Cu) (net 3))
+  (segment (start 183.5 92.6) (end 183.5 90.9) (width 0.6) (layer F.Cu) (net 3))
+  (segment (start 200.94 93.7) (end 184.6 93.7) (width 0.6) (layer F.Cu) (net 3))
+  (segment (start 202.7 91.94) (end 200.94 93.7) (width 0.6) (layer F.Cu) (net 3))
+  (segment (start 183.5 90.9) (end 183.5 83.25) (width 0.6) (layer F.Cu) (net 3))
+  (segment (start 183.5 83.25) (end 183.1 82.85) (width 0.6) (layer F.Cu) (net 3))
+  (segment (start 183.5 73.1) (end 183.5 80.55) (width 0.6) (layer F.Cu) (net 4))
+  (segment (start 183.5 80.55) (end 183.1 80.95) (width 0.6) (layer F.Cu) (net 4))
   (zone (net 1) (net_name Earth) (layer F.Cu) (hatch edge 0.508)
     (connect_pads (clearance 0.3))
@@
     (polygon
       (pts
-        (xy 206.1 68.5) (xy 176.7 68.5) (xy 176.7 95.9) (xy 206.1 95.9)
+        (xy 205.8 70.3) (xy 176.4 70.3) (xy 176.4 95.7) (xy 205.8 95.7)
       )
     )
@@
     (polygon
       (pts
-        (xy 206.1 68.5) (xy 176.7 68.5) (xy 176.7 95.9) (xy 206.1 95.9)
+        (xy 205.7 70.3) (xy 176.3 70.3) (xy 176.3 95.7) (xy 205.7 95.7)
       )
     )
