File: BGP_F1/BUF/BUF.sch (KiCad schematic (older format))
At the start: 20 parts, among them P1 CONN_01X02, P2 CONN_01X05, P3 CONN_01X12, U1 MC33178

Commit message: F boards routed, various optimisations made
Parts:
- removed C1: 0.1u, Capacitors_Tantalum_SMD:TantalC_SizeR_EIA-2012, symbol C_Small
- added C1: 0.01u, Capacitors_Tantalum_SMD:TantalC_SizeR_EIA-2012, symbol CP1_Small
- added C5: 10u, Capacitors_Tantalum_SMD:TantalC_SizeR_EIA-2012, symbol CP1_Small
- R1, R10, R11, R2, R3, R4, R5, R6, R7, R8, R9: footprint Resistors_SMD:R_0805_HandSoldering -> Resistors_SMD:R_0603_HandSoldering
- RV1: footprint Potentiometers:Potentiometer_Trimmer_Bourns_3269X -> Potentiometers:Potentiometer_Trimmer_Bourns_3296X
- U1: footprint Housings_SSOP:MSOP-8_3x3mm_Pitch0.65mm -> Housings_SOIC:SOIC-8_3.9x4.9mm_Pitch1.27mm
Connections:
- net Earth: now also C5.2
- net IN: now also C1.2
- net PG1_1: now also C2.2, P3.11 (P11), P3.12 (P12), R8.1, R9.2, U1.7; no longer R7.1, R8.2
- net PG1_2: now also R10.2, R9.1; no longer C2.2, P3.10 (P10), R8.1, R9.2, U1.7
- net V+: now also C5.1
- net at R3.1, U1.3 (+): now also C1.1
- removed net PG2_2: P3.11 (P11), P3.12 (P12), R10.2, R9.1
- new net PG2_1: P3.10 (P10), R7.1, R8.2
Changed lines of the file:
@@
 F 0 "U1" H 4400 4350 50  0000 L CNN
 F 1 "MC33178" H 4400 3950 50  0000 L CNN
-F 2 "Housings_SSOP:MSOP-8_3x3mm_Pitch0.65mm" H 4300 4200 50  0001 C CNN
+F 2 "Housings_SOIC:SOIC-8_3.9x4.9mm_Pitch1.27mm" H 4300 4200 50  0001 C CNN
 F 3 "" H 4400 4300 50  0000 C CNN
 	1    4400 4150
@@
 V+
 $Comp
-L C_Small C1
-U 1 1 5A5E8958
-P 3800 4250
-F 0 "C1" H 3810 4320 50  0000 L CNN
-F 1 "0.1u" H 3810 4170 50  0000 L CNN
-F 2 "Capacitors_Tantalum_SMD:TantalC_SizeR_EIA-2012" H 3800 4250 50  0001 C CNN
-F 3 "" H 3800 4250 50  0000 C CNN
-	1    3800 4250
-	0    1    1    0
-$EndComp
-$Comp
 L R_Small R3
 U 1 1 5A5E8981
@@
 F 0 "R3" H 4030 4620 50  0000 L CNN
 F 1 "499k" H 4030 4560 50  0000 L CNN
-F 2 "Resistors_SMD:R_0805_HandSoldering" H 4000 4600 50  0001 C CNN
+F 2 "Resistors_SMD:R_0603_HandSoldering" H 4000 4600 50  0001 C CNN
 F 3 "" H 4000 4600 50  0000 C CNN
 	1    4000 4600
@@
 F 0 "R1" H 3580 4620 50  0000 L CNN
 F 1 "499k" H 3580 4560 50  0000 L CNN
-F 2 "Resistors_SMD:R_0805_HandSoldering" H 3550 4600 50  0001 C CNN
+F 2 "Resistors_SMD:R_0603_HandSoldering" H 3550 4600 50  0001 C CNN
 F 3 "" H 3550 4600 50  0000 C CNN
 	1    3550 4600
@@
 F 0 "RV1" H 4000 3470 50  0000 C CNN
 F 1 "POT" H 4000 3550 50  0000 C CNN
-F 2 "Potentiometers:Potentiometer_Trimmer_Bourns_3269X" H 4000 3550 50  0001 C CNN
+F 2 "Potentiometers:Potentiometer_Trimmer_Bourns_3296X" H 4000 3550 50  0001 C CNN
 F 3 "" H 4000 3550 50  0000 C CNN
 	1    4000 3550
@@
 F 0 "R2" H 3730 3570 50  0000 L CNN
 F 1 "2.49k" H 3730 3510 50  0000 L CNN
-F 2 "Resistors_SMD:R_0805_HandSoldering" H 3700 3550 50  0001 C CNN
+F 2 "Resistors_SMD:R_0603_HandSoldering" H 3700 3550 50  0001 C CNN
 F 3 "" H 3700 3550 50  0000 C CNN
 	1    3700 3550
@@
 F 0 "R4" H 4930 4170 50  0000 L CNN
 F 1 "4.99k" H 4930 4110 50  0000 L CNN
-F 2 "Resistors_SMD:R_0805_HandSoldering" H 4900 4150 50  0001 C CNN
+F 2 "Resistors_SMD:R_0603_HandSoldering" H 4900 4150 50  0001 C CNN
 F 3 "" H 4900 4150 50  0000 C CNN
 	1    4900 4150
@@
 F 0 "R5" H 5930 4170 50  0000 L CNN
 F 1 "4.99k" H 5930 4110 50  0000 L CNN
-F 2 "Resistors_SMD:R_0805_HandSoldering" H 5900 4150 50  0001 C CNN
+F 2 "Resistors_SMD:R_0603_HandSoldering" H 5900 4150 50  0001 C CNN
 F 3 "" H 5900 4150 50  0000 C CNN
 	1    5900 4150
@@
 F 0 "U1" H 6300 4250 50  0000 L CNN
 F 1 "MC33178" H 6300 3850 50  0000 L CNN
-F 2 "Housings_SSOP:MSOP-8_3x3mm_Pitch0.65mm" H 6200 4100 50  0001 C CNN
+F 2 "Housings_SOIC:SOIC-8_3.9x4.9mm_Pitch1.27mm" H 6200 4100 50  0001 C CNN
 F 3 "" H 6300 4200 50  0000 C CNN
 	2    6300 4050
@@
 F 0 "R7" H 6230 3420 50  0000 L CNN
 F 1 "15k" H 6230 3360 50  0000 L CNN
-F 2 "Resistors_SMD:R_0805_HandSoldering" H 6200 3400 50  0001 C CNN
+F 2 "Resistors_SMD:R_0603_HandSoldering" H 6200 3400 50  0001 C CNN
 F 3 "" H 6200 3400 50  0000 C CNN
 	1    6200 3400
@@
 F 0 "R6" H 6230 3070 50  0000 L CNN
 F 1 "15k" H 6230 3010 50  0000 L CNN
-F 2 "Resistors_SMD:R_0805_HandSoldering" H 6200 3050 50  0001 C CNN
+F 2 "Resistors_SMD:R_0603_HandSoldering" H 6200 3050 50  0001 C CNN
 F 3 "" H 6200 3050 50  0000 C CNN
 	1    6200 3050
 	0    1    1    0
 $EndComp
-Text Label 6450 3400 1    60   ~ 0
+Text Label 6950 4050 1    60   ~ 0
 PG1_1
-Text Label 6550 3400 1    60   ~ 0
+Text Label 7050 4050 1    60   ~ 0
 PG1_2
-Text Label 6650 3400 1    60   ~ 0
+Text Label 7150 4050 1    60   ~ 0
 PG1_3
 Wire Wire Line
@@
 Text Label 6300 3050 0    60   ~ 0
 Vref
-Text Label 6950 4050 1    60   ~ 0
+Text Label 6450 3400 1    60   ~ 0
 PG2_1
-Text Label 7050 4050 1    60   ~ 0
+Text Label 6550 3400 1    60   ~ 0
 PG2_2
-Text Label 7150 4050 1    60   ~ 0
+Text Label 6650 3400 1    60   ~ 0
 PG2_3
 Connection ~ 6750 4050
@@
 F 0 "R8" H 6530 3520 50  0000 L CNN
 F 1 "20k" H 6530 3460 50  0000 L CNN
-F 2 "Resistors_SMD:R_0805_HandSoldering" H 6500 3500 50  0001 C CNN
+F 2 "Resistors_SMD:R_0603_HandSoldering" H 6500 3500 50  0001 C CNN
 F 3 "" H 6500 3500 50  0000 C CNN
 	1    6500 3500
@@
 F 0 "R9" H 7030 4170 50  0000 L CNN
 F 1 "20k" H 7030 4110 50  0000 L CNN
-F 2 "Resistors_SMD:R_0805_HandSoldering" H 7000 4150 50  0001 C CNN
+F 2 "Resistors_SMD:R_0603_HandSoldering" H 7000 4150 50  0001 C CNN
 F 3 "" H 7000 4150 50  0000 C CNN
 	1    7000 4150
@@
 F 0 "R10" H 7330 4070 50  0000 L CNN
 F 1 "15k" H 7330 4010 50  0000 L CNN
-F 2 "Resistors_SMD:R_0805_HandSoldering" H 7300 4050 50  0001 C CNN
+F 2 "Resistors_SMD:R_0603_HandSoldering" H 7300 4050 50  0001 C CNN
 F 3 "" H 7300 4050 50  0000 C CNN
 	1    7300 4050
@@
 F 0 "R11" H 7530 4270 50  0000 L CNN
 F 1 "15k" H 7530 4210 50  0000 L CNN
-F 2 "Resistors_SMD:R_0805_HandSoldering" H 7500 4250 50  0001 C CNN
+F 2 "Resistors_SMD:R_0603_HandSoldering" H 7500 4250 50  0001 C CNN
 F 3 "" H 7500 4250 50  0000 C CNN
 	1    7500 4250
@@
 Text Label 8550 4650 2    60   ~ 0
 PG2_3
+$Comp
+L CP1_Small C1
+U 1 1 5A5FD792
+P 3800 4250
+F 0 "C1" H 3810 4320 50  0000 L CNN
+F 1 "0.01u" H 3810 4170 50  0000 L CNN
+F 2 "Capacitors_Tantalum_SMD:TantalC_SizeR_EIA-2012" H 3800 4250 50  0001 C CNN
+F 3 "" H 3800 4250 50  0000 C CNN
+	1    3800 4250
+	0    1    1    0
+$EndComp
+$Comp
+L CP1_Small C5
+U 1 1 5A5FDAB4
+P 7800 4600
+F 0 "C5" H 7810 4670 50  0000 L CNN
+F 1 "10u" H 7810 4520 50  0000 L CNN
+F 2 "Capacitors_Tantalum_SMD:TantalC_SizeR_EIA-2012" H 7800 4600 50  0001 C CNN
+F 3 "" H 7800 4600 50  0000 C CNN
+	1    7800 4600
+	1    0    0    -1
+$EndComp
+$Comp
+L Earth #PWR06
+U 1 1 5A5FDB44
+P 7800 4700
+F 0 "#PWR06" H 7800 4450 50  0001 C CNN
+F 1 "Earth" H 7800 4550 50  0001 C CNN
+F 2 "" H 7800 4700 50  0000 C CNN
+F 3 "" H 7800 4700 50  0000 C CNN
+	1    7800 4700
+	1    0    0    -1
+$EndComp
+Text Label 7800 4500 1    60   ~ 0
+V+
 $EndSCHEMATC

Commit message: Pot tinkering
Connections:
- net PF1_1: no longer P3.2 (P2), R4.1
- net PF1_3: no longer P3.4 (P4)
- net PG1_1: no longer P3.12 (P12)
- net PG1_2: no longer P3.9 (P9)
- new net PF1_2: P3.2 (P2), R4.1
- new net PF2_1: P3.4 (P4)
- new net PG1_3: P3.9 (P9)
- new net PG2_3: P3.12 (P12)
Changed lines of the file:
@@
 LIBS:contrib
 LIBS:valves
+LIBS:BUF-cache
 EELAYER 25 0
 EELAYER END
@@
 	0    1    1    0
 $EndComp
-Text Label 5100 4150 1    60   ~ 0
-PF1_1
 Text Label 5200 4150 1    60   ~ 0
 PF1_2
@@
 Wire Wire Line
 	5200 4150 5000 4150
-Text Label 5550 4150 1    60   ~ 0
-PF2_1
 Text Label 5650 4150 1    60   ~ 0
 PF2_2
@@
 Text Label 7050 4050 1    60   ~ 0
 PG1_2
-Text Label 7150 4050 1    60   ~ 0
-PG1_3
 Wire Wire Line
 	6550 3400 6750 3400
@@
 Text Label 6550 3400 1    60   ~ 0
 PG2_2
-Text Label 6650 3400 1    60   ~ 0
-PG2_3
 Connection ~ 6750 4050
 Wire Wire Line

Commit message: New F0 Version
Parts:
- P2: footprint Connectors_Molex:Molex_MicroLatch-53253-0570_05x2.00mm_Straight -> Connectors_JST:JST_PH_B5B-PH-K_05x2.00mm_Straight
Changed lines of the file:
@@
 EESchema Schematic File Version 2
+LIBS:BUF-rescue
 LIBS:power
 LIBS:device
@@
 F 0 "P2" H 2600 4450 50  0000 C CNN
 F 1 "CONN_01X05" V 2700 4150 50  0000 C CNN
-F 2 "Connectors_Molex:Molex_MicroLatch-53253-0570_05x2.00mm_Straight" H 2600 4150 50  0001 C CNN
+F 2 "Connectors_JST:JST_PH_B5B-PH-K_05x2.00mm_Straight" H 2600 4150 50  0001 C CNN
 F 3 "" H 2600 4150 50  0000 C CNN
 	1    2600 4150

Commit message: F1 updates to reverse pots
Parts:
- R1, R3: value 499k -> 470k
- R10, R11, R6, R7: value 15k -> 27k
- R2: value 2.49k -> 2.4k
- R4, R5: value 4.99k -> 4.7k
Connections:
- net PF1_1: now also P3.7 (P7); no longer P3.1 (P1)
- net PF1_2: now also P3.8 (P8); no longer P3.2 (P2)
- net PF1_3: now also P3.11 (P11), P3.9 (P9); no longer P3.3 (P3), P3.5 (P5)
- net PF2_1: now also P3.10 (P10); no longer P3.4 (P4)
- net PF3_3: now also P3.12 (P12); no longer P3.6 (P6)
- net PG1_1: now also P3.1 (P1), P3.5 (P5); no longer P3.11 (P11), P3.7 (P7)
- net PG1_2: now also P3.2 (P2); no longer P3.8 (P8)
- net PG1_3: now also P3.3 (P3); no longer P3.9 (P9)
- net PG2_1: now also P3.4 (P4); no longer P3.10 (P10)
- net PG2_3: now also P3.6 (P6); no longer P3.12 (P12)
Changed lines of the file:
@@
 P 4000 4600
 F 0 "R3" H 4030 4620 50  0000 L CNN
-F 1 "499k" H 4030 4560 50  0000 L CNN
+F 1 "470k" H 4030 4560 50  0000 L CNN
 F 2 "Resistors_SMD:R_0603_HandSoldering" H 4000 4600 50  0001 C CNN
 F 3 "" H 4000 4600 50  0000 C CNN
@@
 P 3550 4600
 F 0 "R1" H 3580 4620 50  0000 L CNN
-F 1 "499k" H 3580 4560 50  0000 L CNN
+F 1 "470k" H 3580 4560 50  0000 L CNN
 F 2 "Resistors_SMD:R_0603_HandSoldering" H 3550 4600 50  0001 C CNN
 F 3 "" H 3550 4600 50  0000 C CNN
@@
 P 3700 3550
 F 0 "R2" H 3730 3570 50  0000 L CNN
-F 1 "2.49k" H 3730 3510 50  0000 L CNN
+F 1 "2.4k" H 3730 3510 50  0000 L CNN
 F 2 "Resistors_SMD:R_0603_HandSoldering" H 3700 3550 50  0001 C CNN
 F 3 "" H 3700 3550 50  0000 C CNN
@@
 P 4900 4150
 F 0 "R4" H 4930 4170 50  0000 L CNN
-F 1 "4.99k" H 4930 4110 50  0000 L CNN
+F 1 "4.7k" H 4930 4110 50  0000 L CNN
 F 2 "Resistors_SMD:R_0603_HandSoldering" H 4900 4150 50  0001 C CNN
 F 3 "" H 4900 4150 50  0000 C CNN
@@
 P 5900 4150
 F 0 "R5" H 5930 4170 50  0000 L CNN
-F 1 "4.99k" H 5930 4110 50  0000 L CNN
+F 1 "4.7k" H 5930 4110 50  0000 L CNN
 F 2 "Resistors_SMD:R_0603_HandSoldering" H 5900 4150 50  0001 C CNN
 F 3 "" H 5900 4150 50  0000 C CNN
@@
 P 6200 3400
 F 0 "R7" H 6230 3420 50  0000 L CNN
-F 1 "15k" H 6230 3360 50  0000 L CNN
+F 1 "27k" H 6230 3360 50  0000 L CNN
 F 2 "Resistors_SMD:R_0603_HandSoldering" H 6200 3400 50  0001 C CNN
 F 3 "" H 6200 3400 50  0000 C CNN
@@
 P 6200 3050
 F 0 "R6" H 6230 3070 50  0000 L CNN
-F 1 "15k" H 6230 3010 50  0000 L CNN
+F 1 "27k" H 6230 3010 50  0000 L CNN
 F 2 "Resistors_SMD:R_0603_HandSoldering" H 6200 3050 50  0001 C CNN
 F 3 "" H 6200 3050 50  0000 C CNN
@@
 P 7300 4050
 F 0 "R10" H 7330 4070 50  0000 L CNN
-F 1 "15k" H 7330 4010 50  0000 L CNN
+F 1 "27k" H 7330 4010 50  0000 L CNN
 F 2 "Resistors_SMD:R_0603_HandSoldering" H 7300 4050 50  0001 C CNN
 F 3 "" H 7300 4050 50  0000 C CNN
@@
 P 7500 4250
 F 0 "R11" H 7530 4270 50  0000 L CNN
-F 1 "15k" H 7530 4210 50  0000 L CNN
+F 1 "27k" H 7530 4210 50  0000 L CNN
 F 2 "Resistors_SMD:R_0603_HandSoldering" H 7500 4250 50  0001 C CNN
 F 3 "" H 7500 4250 50  0000 C CNN
@@
 	1    0    0    -1
 $EndComp
+Text Label 8550 4150 2    60   ~ 0
+PF1_1
+Text Label 8550 4250 2    60   ~ 0
+PF1_2
+Text Label 8550 4350 2    60   ~ 0
+PF1_3
+Wire Wire Line
+	5400 4500 5400 4150
+Wire Wire Line
+	5400 4700 5400 4950
+Wire Wire Line
+	5400 4950 6750 4950
+Text Label 8550 4450 2    60   ~ 0
+PF2_1
+Text Label 8550 4550 2    60   ~ 0
+PF2_2
+Text Label 8550 4650 2    60   ~ 0
+PF3_3
 Text Label 8550 3550 2    60   ~ 0
-PF1_1
+PG1_1
 Text Label 8550 3650 2    60   ~ 0
-PF1_2
+PG1_2
 Text Label 8550 3750 2    60   ~ 0
-PF1_3
-Wire Wire Line
-	5400 4500 5400 4150
-Wire Wire Line
-	5400 4700 5400 4950
-Wire Wire Line
-	5400 4950 6750 4950
+PG1_3
 Text Label 8550 3850 2    60   ~ 0
-PF2_1
+PG2_1
 Text Label 8550 3950 2    60   ~ 0
-PF2_2
+PG2_2
 Text Label 8550 4050 2    60   ~ 0
-PF3_3
-Text Label 8550 4150 2    60   ~ 0
-PG1_1
-Text Label 8550 4250 2    60   ~ 0
-PG1_2
-Text Label 8550 4350 2    60   ~ 0
-PG1_3
-Text Label 8550 4450 2    60   ~ 0
-PG2_1
-Text Label 8550 4550 2    60   ~ 0
-PG2_2
-Text Label 8550 4650 2    60   ~ 0
 PG2_3
 $Comp
