File: BGP_F1/HPF/HPF.kicad_pcb (KiCad board)
At the start: 2 copper layers, 30 x 24 mm, 15 parts, among them P1 CONN_01X05, P2 CONN_01X06, U1 MC33178

Commit message: Flipped boards so that they should be facing the right way
Parts:
- P1: moved to F.Cu
Connections:
- C1 pad 1: /VF_1 -> /VF_2
- P2 pad 2: /VF_1 -> /VF_2
- P2 pad 6: /VG_2 -> /VG_3
- U1 pad 3: /VF_1 -> /VF_2
Routing:
- net /VF_2: track 0.00 -> 28.6 mm, vias 0 -> 1
- net /VF_1: track 28.6 -> 0.95 mm, vias 1 -> 0

Commit message: Pot tinkering
Connections:
- C2 pad 1: /VG_2 -> /VG_3
- C2 pad 2: /VG_1 -> /VG_2
- R3 pad 2: /VG_1 -> /VG_2
- R4 pad 1: /VG_2 -> /VG_3
- R4 pad 2: /VG_1 -> /VG_2
- R5 pad 2: /VG_2 -> /VG_3
- R6 pad 2: /VG_2 -> /VG_3
- U1 pad 1: /VG_2 -> /VG_3
- U1 pad 2: /VG_1 -> /VG_2
Routing:
- net /VG_3: track 0.00 -> 27.3 mm, vias 0 -> 2
- net /VG_1: track 18.5 -> 0.00 mm
- net /VG_2: track 27.2 -> 23.0 mm, vias 2 -> 0
- net /VF_1: track 0.95 -> 0.00 mm

Commit message: New F0 Version
Parts:
- P1: footprint Connectors_Molex:Molex_MicroLatch-53253-0570_05x2.00mm_Straight -> Connectors_JST:JST_PH_B5B-PH-K_05x2.00mm_Straight
- moved P1 0.40 mm to (162.0, 108.4)
Changed lines of the file:
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@@
     (add_net Earth)
+  )
+  (module Connectors_JST:JST_PH_B5B-PH-K_05x2.00mm_Straight (layer F.Cu)
+    (at 162 108.4 180)
+    (descr "JST PH series connector, B5B-PH-K, top entry type, through hole, Datasheet: http://www.jst-mfg.com/product/pdf/eng/ePH.pdf")
+    (tags "connector jst ph")
+    (fp_text reference P1 (at 10.8 2.5 180) (layer F.SilkS)
+      (effects (font (size 0.6 0.6) (thickness 0.15)))
+    )
+    (fp_text value CONN_01X05 (at 4 3.8 180) (layer F.Fab) hide
+      (effects (font (size 0.6 0.6) (thickness 0.15)))
+    )
+    (fp_line (start -2.05 -1.8) (end -2.05 2.9) (layer F.SilkS) (width 0.12))
+    (fp_line (start -2.05 2.9) (end 10.05 2.9) (layer F.SilkS) (width 0.12))
+    (fp_line (start 10.05 2.9) (end 10.05 -1.8) (layer F.SilkS) (width 0.12))
+    (fp_line (start 10.05 -1.8) (end -2.05 -1.8) (layer F.SilkS) (width 0.12))
+    (fp_line (start 0.5 -1.8) (end 0.5 -1.2) (layer F.SilkS) (width 0.12))
+    (fp_line (start 0.5 -1.2) (end -1.45 -1.2) (layer F.SilkS) (width 0.12))
+    (fp_line (start -1.45 -1.2) (end -1.45 2.3) (layer F.SilkS) (width 0.12))
+    (fp_line (start -1.45 2.3) (end 9.45 2.3) (layer F.SilkS) (width 0.12))
+    (fp_line (start 9.45 2.3) (end 9.45 -1.2) (layer F.SilkS) (width 0.12))
+    (fp_line (start 9.45 -1.2) (end 7.5 -1.2) (layer F.SilkS) (width 0.12))
+    (fp_line (start 7.5 -1.2) (end 7.5 -1.8) (layer F.SilkS) (width 0.12))
+    (fp_line (start -2.05 -0.5) (end -1.45 -0.5) (layer F.SilkS) (width 0.12))
+    (fp_line (start -2.05 0.8) (end -1.45 0.8) (layer F.SilkS) (width 0.12))
+    (fp_line (start 10.05 -0.5) (end 9.45 -0.5) (layer F.SilkS) (width 0.12))
+    (fp_line (start 10.05 0.8) (end 9.45 0.8) (layer F.SilkS) (width 0.12))
+    (fp_line (start -0.3 -1.8) (end -0.3 -2) (layer F.SilkS) (width 0.12))
+    (fp_line (start -0.3 -2) (end -0.6 -2) (layer F.SilkS) (width 0.12))
+    (fp_line (start -0.6 -2) (end -0.6 -1.8) (layer F.SilkS) (width 0.12))
+    (fp_line (start -0.3 -1.9) (end -0.6 -1.9) (layer F.SilkS) (width 0.12))
+    (fp_line (start 0.9 2.3) (end 0.9 1.8) (layer F.SilkS) (width 0.12))
+    (fp_line (start 0.9 1.8) (end 1.1 1.8) (layer F.SilkS) (width 0.12))
+    (fp_line (start 1.1 1.8) (end 1.1 2.3) (layer F.SilkS) (width 0.12))
+    (fp_line (start 1 2.3) (end 1 1.8) (layer F.SilkS) (width 0.12))
+    (fp_line (start 2.9 2.3) (end 2.9 1.8) (layer F.SilkS) (width 0.12))
+    (fp_line (start 2.9 1.8) (end 3.1 1.8) (layer F.SilkS) (width 0.12))
+    (fp_line (start 3.1 1.8) (end 3.1 2.3) (layer F.SilkS) (width 0.12))
+    (fp_line (start 3 2.3) (end 3 1.8) (layer F.SilkS) (width 0.12))
+    (fp_line (start 4.9 2.3) (end 4.9 1.8) (layer F.SilkS) (width 0.12))
+    (fp_line (start 4.9 1.8) (end 5.1 1.8) (layer F.SilkS) (width 0.12))
+    (fp_line (start 5.1 1.8) (end 5.1 2.3) (layer F.SilkS) (width 0.12))
+    (fp_line (start 5 2.3) (end 5 1.8) (layer F.SilkS) (width 0.12))
+    (fp_line (start 6.9 2.3) (end 6.9 1.8) (layer F.SilkS) (width 0.12))
+    (fp_line (start 6.9 1.8) (end 7.1 1.8) (layer F.SilkS) (width 0.12))
+    (fp_line (start 7.1 1.8) (end 7.1 2.3) (layer F.SilkS) (width 0.12))
+    (fp_line (start 7 2.3) (end 7 1.8) (layer F.SilkS) (width 0.12))
+    (fp_line (start -1.1 -2.1) (end -2.35 -2.1) (layer F.SilkS) (width 0.12))
+    (fp_line (start -2.35 -2.1) (end -2.35 -0.85) (layer F.SilkS) (width 0.12))
+    (fp_line (start -1.1 -2.1) (end -2.35 -2.1) (layer F.Fab) (width 0.1))
+    (fp_line (start -2.35 -2.1) (end -2.35 -0.85) (layer F.Fab) (width 0.1))
+    (fp_line (start -1.95 -1.7) (end -1.95 2.8) (layer F.Fab) (width 0.1))
+    (fp_line (start -1.95 2.8) (end 9.95 2.8) (layer F.Fab) (width 0.1))
+    (fp_line (start 9.95 2.8) (end 9.95 -1.7) (layer F.Fab) (width 0.1))
+    (fp_line (start 9.95 -1.7) (end -1.95 -1.7) (layer F.Fab) (width 0.1))
+    (fp_line (start -2.45 -2.2) (end -2.45 3.3) (layer F.CrtYd) (width 0.05))
+    (fp_line (start -2.45 3.3) (end 10.45 3.3) (layer F.CrtYd) (width 0.05))
+    (fp_line (start 10.45 3.3) (end 10.45 -2.2) (layer F.CrtYd) (width 0.05))
+    (fp_line (start 10.45 -2.2) (end -2.45 -2.2) (layer F.CrtYd) (width 0.05))
+    (fp_text user %R (at 4 1.5 180) (layer F.Fab) hide
+      (effects (font (size 0.6 0.6) (thickness 0.15)))
+    )
+    (pad 1 thru_hole rect (at 0 0 180) (size 1.2 1.7) (drill 0.75) (layers *.Cu *.Mask)
+      (net 10 Earth))
+    (pad 2 thru_hole oval (at 2 0 180) (size 1.2 1.7) (drill 0.75) (layers *.Cu *.Mask)
+      (net 11 /BUF_I))
+    (pad 3 thru_hole oval (at 4 0 180) (size 1.2 1.7) (drill 0.75) (layers *.Cu *.Mask)
+      (net 8 /OUT))
+    (pad 4 thru_hole oval (at 6 0 180) (size 1.2 1.7) (drill 0.75) (layers *.Cu *.Mask)
+      (net 6 /Vref))
+    (pad 5 thru_hole oval (at 8 0 180) (size 1.2 1.7) (drill 0.75) (layers *.Cu *.Mask)
+      (net 9 /V+))
+    (model ${KISYS3DMOD}/Connectors_JST.3dshapes/JST_PH_B5B-PH-K_05x2.00mm_Straight.wrl
+      (at (xyz 0 0 0))
+      (scale (xyz 1 1 1))
+      (rotate (xyz 0 0 0))
+    )
   )
   (module LIBS:Potentiometer_Alpha_Double_Vertical_Dual_Shaft (layer B.Cu)
@@
       (net 10 Earth))
     (model Capacitors_Tantalum_SMD.3dshapes/TantalC_SizeR_EIA-2012.wrl
-      (at (xyz 0 0 0))
-      (scale (xyz 1 1 1))
-      (rotate (xyz 0 0 0))
-    )
-  )
-  (module Connectors_Molex:Molex_MicroLatch-53253-0570_05x2.00mm_Straight (layer F.Cu)
-    (at 162 108 180)
-    (descr "Molex Micro-Latch connector, PN:53253-0570, top entry type, through hole")
-    (tags "conn molex micro latch")
-    (fp_text reference P1 (at -1.7 -2.3 180) (layer F.SilkS)
-      (effects (font (size 0.6 0.6) (thickness 0.15)))
-    )
-    (fp_text value CONN_01X05 (at 4 -3.5 180) (layer F.Fab) hide
-      (effects (font (size 0.6 0.6) (thickness 0.15)))
-    )
-    (fp_line (start -2.6 -2.1) (end -2.6 2.75) (layer F.CrtYd) (width 0.05))
-    (fp_line (start -2.6 2.75) (end 10.55 2.75) (layer F.CrtYd) (width 0.05))
-    (fp_line (start 10.55 2.75) (end 10.55 -2.1) (layer F.CrtYd) (width 0.05))
-    (fp_line (start 10.55 -2.1) (end -2.6 -2.1) (layer F.CrtYd) (width 0.05))
-    (fp_line (start -2.1 -1.6) (end -2.1 2.25) (layer F.SilkS) (width 0.15))
-    (fp_line (start -2.1 2.25) (end 10.1 2.25) (layer F.SilkS) (width 0.15))
-    (fp_line (start 10.1 2.25) (end 10.1 -1.6) (layer F.SilkS) (width 0.15))
-    (fp_line (start 10.1 -1.6) (end -2.1 -1.6) (layer F.SilkS) (width 0.15))
-    (fp_line (start 0 -2) (end -0.3 -2.6) (layer F.SilkS) (width 0.15))
-    (fp_line (start -0.3 -2.6) (end 0.3 -2.6) (layer F.SilkS) (width 0.15))
-    (fp_line (start 0.3 -2.6) (end 0 -2) (layer F.SilkS) (width 0.15))
-    (fp_line (start -2.1 0.8) (end -1.7 0.8) (layer F.SilkS) (width 0.15))
-    (fp_line (start 10.1 0.8) (end 9.7 0.8) (layer F.SilkS) (width 0.15))
-    (fp_line (start 4 -1.2) (end -1.7 -1.2) (layer F.SilkS) (width 0.15))
-    (fp_line (start -1.7 -1.2) (end -1.7 0) (layer F.SilkS) (width 0.15))
-    (fp_line (start -1.7 0) (end -1.3 0) (layer F.SilkS) (width 0.15))
-    (fp_line (start -1.3 0) (end -1.3 0.4) (layer F.SilkS) (width 0.15))
-    (fp_line (start -1.3 0.4) (end -1.7 0.4) (layer F.SilkS) (width 0.15))
-    (fp_line (start -1.7 0.4) (end -1.7 2.25) (layer F.SilkS) (width 0.15))
-    (fp_line (start 4 -1.2) (end 9.7 -1.2) (layer F.SilkS) (width 0.15))
-    (fp_line (start 9.7 -1.2) (end 9.7 0) (layer F.SilkS) (width 0.15))
-    (fp_line (start 9.7 0) (end 9.3 0) (layer F.SilkS) (width 0.15))
-    (fp_line (start 9.3 0) (end 9.3 0.4) (layer F.SilkS) (width 0.15))
-    (fp_line (start 9.3 0.4) (end 9.7 0.4) (layer F.SilkS) (width 0.15))
-    (fp_line (start 9.7 0.4) (end 9.7 2.25) (layer F.SilkS) (width 0.15))
-    (pad 1 thru_hole rect (at 0 0 180) (size 1.5 1.5) (drill 0.8) (layers *.Cu *.Mask)
-      (net 10 Earth))
-    (pad 2 thru_hole circle (at 2 0 180) (size 1.5 1.5) (drill 0.8) (layers *.Cu *.Mask)
-      (net 11 /BUF_I))
-    (pad 3 thru_hole circle (at 4 0 180) (size 1.5 1.5) (drill 0.8) (layers *.Cu *.Mask)
-      (net 8 /OUT))
-    (pad 4 thru_hole circle (at 6 0 180) (size 1.5 1.5) (drill 0.8) (layers *.Cu *.Mask)
-      (net 6 /Vref))
-    (pad 5 thru_hole circle (at 8 0 180) (size 1.5 1.5) (drill 0.8) (layers *.Cu *.Mask)
-      (net 9 /V+))
-    (model Connectors_Molex.3dshapes/Molex_MicroLatch-53253-0570_05x2.00mm_Straight.wrl
       (at (xyz 0 0 0))
       (scale (xyz 1 1 1))
@@
   (segment (start 162 108) (end 162 106.95) (width 0.5) (layer B.Cu) (net 10) (status 10))
   (segment (start 162 106.95) (end 156.82398 101.77398) (width 0.5) (layer B.Cu) (net 10))
-  (segment (start 144.9 105) (end 149.5 109.6) (width 0.5) (layer B.Cu) (net 11))
-  (segment (start 149.5 109.6) (end 159.5 109.6) (width 0.5) (layer B.Cu) (net 11))
-  (segment (start 159.5 109.6) (end 160 109.1) (width 0.5) (layer B.Cu) (net 11))
-  (segment (start 160 109.1) (end 160 108) (width 0.5) (layer B.Cu) (net 11) (status 20))
+  (segment (start 144.9 105) (end 150.1 110.2) (width 0.5) (layer B.Cu) (net 11))
+  (segment (start 150.1 110.2) (end 158.9 110.2) (width 0.5) (layer B.Cu) (net 11))
+  (segment (start 158.9 110.2) (end 160 109.1) (width 0.5) (layer B.Cu) (net 11))
+  (segment (start 160 109.1) (end 160 108) (width 0.5) (layer B.Cu) (net 11))
   (segment (start 144.9 104) (end 144.9 105) (width 0.5) (layer F.Cu) (net 11) (status 10))
   (via (at 144.9 105) (size 0.6) (drill 0.4) (layers F.Cu B.Cu) (net 11))

Commit message: F1 updates to reverse pots
Parts:
- C3: value 39n -> 22n
- R3, R5, R7: value 4.99k -> 4.7k
- R4: value 24.9k -> 24k
- R6: value 49.9k -> 47k
Changed lines of the file:
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@@
       (effects (font (size 0.6 0.6) (thickness 0.15)))
     )
-    (fp_text value 39n (at 0 2.3 180) (layer F.Fab) hide
+    (fp_text value 22n (at 0 2.3 180) (layer F.Fab) hide
       (effects (font (size 0.6 0.6) (thickness 0.15)))
     )
@@
       (effects (font (size 0.6 0.6) (thickness 0.15)))
     )
-    (fp_text value 4.99k (at 0 1.9) (layer F.Fab) hide
+    (fp_text value 4.7k (at 0 1.9) (layer F.Fab) hide
       (effects (font (size 0.6 0.6) (thickness 0.15)))
     )
@@
       (effects (font (size 0.6 0.6) (thickness 0.15)))
     )
-    (fp_text value 24.9k (at 0 1.9 180) (layer F.Fab) hide
+    (fp_text value 24k (at 0 1.9 180) (layer F.Fab) hide
       (effects (font (size 0.6 0.6) (thickness 0.15)))
     )
@@
       (effects (font (size 0.6 0.6) (thickness 0.15)))
     )
-    (fp_text value 4.99k (at 0 1.9 180) (layer F.Fab) hide
+    (fp_text value 4.7k (at 0 1.9 180) (layer F.Fab) hide
       (effects (font (size 0.6 0.6) (thickness 0.15)))
     )
@@
       (effects (font (size 0.6 0.6) (thickness 0.15)))
     )
-    (fp_text value 49.9k (at 0 1.9) (layer F.Fab) hide
+    (fp_text value 47k (at 0 1.9) (layer F.Fab) hide
       (effects (font (size 0.6 0.6) (thickness 0.15)))
     )
@@
       (effects (font (size 0.6 0.6) (thickness 0.15)))
     )
-    (fp_text value 4.99k (at 0 1.9 270) (layer F.Fab) hide
-      (effects (font (size 0.6 0.6) (thickness 0.15)))
-    )
+    (fp_text value 4.7k (at 0 1.9 270) (layer F.Fab) hide
+      (effects (font (size 0.6 0.6) (thickness 0.15)))
+    )

Commit message: HPF Done
Parts:
- removed C3: 22n, Capacitors_SMD:C_1206_HandSoldering
- C1, C2: footprint Capacitors_SMD:C_0805_HandSoldering -> Capacitors_SMD:C_0805
- P1: moved to B.Cu
- P2: footprint LIBS:Potentiometer_Alpha_Double_Vertical_Dual_Shaft -> LIBS:Potentiometer_Alps_RK097_Double_Vertical_Dual_Shaft
- R1, R2, R3, R4, R5, R6, R7: footprint Resistors_SMD:R_0603_HandSoldering -> Resistors_SMD:R_0603
- moved R2 13.0 mm to (151.0, 89.0)
- moved C1 9.81 mm to (151.5, 94.2)
- moved C4 9.66 mm to (164.9, 95.8), turned to 180 degrees
- moved R1 8.68 mm to (151.0, 96.9), turned to 0 degrees
- moved R3 6.73 mm to (151.0, 91.5)
- moved R5 6.54 mm to (164.0, 103.6)
- moved C2 3.62 mm to (151.4, 99.6), turned to 0 degrees
- moved R7 3.40 mm to (164.0, 98.6), turned to 0 degrees
- moved R4 3.30 mm to (150.9, 102.3), turned to 0 degrees
- moved P1 2.40 mm to (162.0, 106.0)
- moved P2 1.66 mm to (155.5, 90.0)
- moved R6 1.00 mm to (164.0, 101.1)
- moved C5 1.00 mm to (158.0, 100.0), turned to 180 degrees
- moved U1 0.40 mm to (158.0, 99.4)
Routing:
- net /Vref: track 8.52 -> 24.4 mm, vias 2 -> 0
- net /VF_3: track 24.8 -> 10.0 mm, vias 1 -> 0
- net /VF_2: track 28.6 -> 15.1 mm, vias 1 -> 2
- net Net-(C4-Pad1): track 18.7 -> 5.61 mm
- net /V+: track 1.62 -> 13.3 mm
- net /OUT: track 13.2 -> 18.8 mm
- net Earth: track 12.7 -> 16.6 mm, vias 1 -> 0
- net Net-(C3-Pad1): track 6.28 -> 2.63 mm
- net /VG_2: track 23.0 -> 20.4 mm
- net Net-(R5-Pad1): track 12.7 -> 10.2 mm
- net /VG_3: track 27.3 -> 27.9 mm
Other:
- board size 30 x 24 mm -> 19 x 22.5 mm
