File: BGP_F0/BUF_v2/BUF.kicad_pcb (KiCad board)
At the start: 2 copper layers, 32 x 26 mm, 33 parts, among them P1 CONN_01X02, P2 CONN_01X02, P3 CONN_01X03, P4 CONN_01X02, P5 CONN_01X09, P6 CONN_01X05, P7 CONN_01X02, Q1 2N5457, Q2 2N5457, U1 MC33178

Commit message: Slight changes
Parts:
- moved P5 0.61 mm to (146.2, 80.5)
Routing:
- net Earth: track 14.5 -> 13.9 mm
- net /PV_2: track 31.0 -> 30.4 mm
- net /PB1_1: track 17.7 -> 17.1 mm
