File: BGP_F0/VOL/VOL.kicad_pcb (KiCad board)
At the start: 2 copper layers, 20 x 26 mm, 4 parts, among them J1 Conn_01x03_Female, J2 Conn_01x03_Female, P1 CONN_01X02

Commit message: Mods and gerbers done
Parts:
- moved RV1 2.00 mm to (145.5, 82.0)
- moved J1 1.00 mm to (150.5, 89.0)
Routing:
- net /VOL_1: track 22.7 -> 20.6 mm
- net /VOL_3: track 12.0 -> 11.0 mm
Changed lines of the file:
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@@
-(kicad_pcb (version 4) (host pcbnew 4.0.7)
+(kicad_pcb (version 4) (host pcbnew 4.0.4-1.fc24-product)
   (general
     (links 6)
-    (no_connects 4)
-    (area 137.924999 75.924999 158.075001 102.075001)
+    (no_connects 0)
+    (area 137.924999 75.174999 158.075001 102.075001)
     (thickness 1.6)
     (drawings 8)
-    (tracks 17)
+    (tracks 14)
     (zones 0)
     (modules 4)
@@
     (visible_elements 7FFFFFFF)
     (pcbplotparams
-      (layerselection 0x00030_80000001)
-      (usegerberextensions false)
+      (layerselection 0x010fc_80000001)
+      (usegerberextensions true)
       (excludeedgelayer true)
       (linewidth 0.100000)
@@
       (outputformat 1)
       (mirror false)
-      (drillshape 1)
+      (drillshape 0)
       (scaleselection 1)
-      (outputdirectory ""))
+      (outputdirectory ../../GERBER/F0_VOL/))
   )
   (net 0 "")
@@
   )
   (module Pin_Headers:Pin_Header_Straight_1x03_Pitch2.54mm (layer B.Cu)
-    (at 150.54 88 90)
+    (at 150.54 89 90)
     (descr "Through hole straight pin header, 1x03, 2.54mm pitch, single row")
     (tags "Through hole pin header THT 1x03 2.54mm single row")
@@
   )
   (module LIBS:Potentiometer_Alps_RK097_Double_Vertical (layer B.Cu)
-    (at 145.5 80 90)
+    (at 145.5 82 90)
     (descr "Potentiometer, vertically mounted, Omeg PC16PU, Omeg PC16PU, Omeg PC16PU, Vishay/Spectrol 248GJ/249GJ Single, Vishay/Spectrol 248GJ/249GJ Single, Vishay/Spectrol 248GJ/249GJ Single, Vishay/Spectrol 248GH/249GH Single, Vishay/Spectrol 148/149 Single, Vishay/Spectrol 148/149 Single, Vishay/Spectrol 148/149 Single, Vishay/Spectrol 148A/149A Single with mounting plates, Vishay/Spectrol 148/149 Double, Vishay/Spectrol 148A/149A Double with mounting plates, Piher PC-16 Single, Piher PC-16 Single, Piher PC-16 Single, Piher PC-16SV Single, Piher PC-16 Double, Piher PC-16 Triple, Piher T16H Single, Piher T16L Single, Piher T16H Double, Alps RK163 Single, Alps RK163 Double, Alps RK097 Single, Alps RK097 Double, http://www.alps.com/prod/info/E/HTML/Potentiometer/RotaryPotentiometers/RK097/RK09712100AV.html")
     (tags "Potentiometer vertical  Omeg PC16PU  Omeg PC16PU  Omeg PC16PU  Vishay/Spectrol 248GJ/249GJ Single  Vishay/Spectrol 248GJ/249GJ Single  Vishay/Spectrol 248GJ/249GJ Single  Vishay/Spectrol 248GH/249GH Single  Vishay/Spectrol 148/149 Single  Vishay/Spectrol 148/149 Single  Vishay/Spectrol 148/149 Single  Vishay/Spectrol 148A/149A Single with mounting plates  Vishay/Spectrol 148/149 Double  Vishay/Spectrol 148A/149A Double with mounting plates  Piher PC-16 Single  Piher PC-16 Single  Piher PC-16 Single  Piher PC-16SV Single  Piher PC-16 Double  Piher PC-16 Triple  Piher T16H Single  Piher T16L Single  Piher T16H Double  Alps RK163 Single  Alps RK163 Double  Alps RK097 Single  Alps RK097 Double")
@@
   (gr_line (start 138 76) (end 138 102) (layer Edge.Cuts) (width 0.15))
   (gr_line (start 158 76) (end 138 76) (layer Edge.Cuts) (width 0.15))
-  (segment (start 143 95.85) (end 143 82.5) (width 0.75) (layer F.Cu) (net 1))
-  (segment (start 143 82.5) (end 145.5 80) (width 0.75) (layer F.Cu) (net 1))
+  (segment (start 142.3 95.15) (end 142.3 85.2) (width 0.75) (layer F.Cu) (net 1))
+  (segment (start 142.3 85.2) (end 145.5 82) (width 0.75) (layer F.Cu) (net 1))
   (segment (start 147 98.5) (end 145.65 98.5) (width 0.75) (layer F.Cu) (net 1))
-  (segment (start 145.65 98.5) (end 143 95.85) (width 0.75) (layer F.Cu) (net 1))
-  (segment (start 147 98.5) (end 147 98.25) (width 0.75) (layer F.Cu) (net 1))
-  (segment (start 147 98.5) (end 146.7 98.2) (width 0.75) (layer F.Cu) (net 1))
-  (segment (start 145.46 92.5) (end 145.46 88) (width 0.75) (layer F.Cu) (net 2))
-  (segment (start 149 98.5) (end 149 96.04) (width 0.75) (layer F.Cu) (net 2))
-  (segment (start 149 96.04) (end 145.46 92.5) (width 0.75) (layer F.Cu) (net 2))
-  (segment (start 150.54 88) (end 150.54 86.4) (width 0.75) (layer F.Cu) (net 3))
-  (segment (start 150.54 86.4) (end 152.3 84.64) (width 0.75) (layer F.Cu) (net 3))
-  (segment (start 152.3 84.64) (end 152.3 81.8) (width 0.75) (layer F.Cu) (net 3))
-  (segment (start 152.3 81.8) (end 151.399999 80.899999) (width 0.75) (layer F.Cu) (net 3))
-  (segment (start 151.399999 80.899999) (end 150.5 80) (width 0.75) (layer F.Cu) (net 3))
-  (segment (start 150.54 92.5) (end 150.54 88) (width 0.75) (layer F.Cu) (net 3))
-  (segment (start 150.5 80) (end 148 80) (width 0.75) (layer F.Cu) (net 3))
-  (segment (start 150.54 80.04) (end 150.5 80) (width 0.75) (layer F.Cu) (net 3))
+  (segment (start 145.65 98.5) (end 142.3 95.15) (width 0.75) (layer F.Cu) (net 1))
+  (segment (start 145.46 92.5) (end 149 96.04) (width 0.75) (layer F.Cu) (net 2))
+  (segment (start 149 96.04) (end 149 98.5) (width 0.75) (layer F.Cu) (net 2))
+  (segment (start 145.46 92.5) (end 145.46 89) (width 0.75) (layer F.Cu) (net 2))
+  (segment (start 150.5 82) (end 148 82) (width 0.75) (layer F.Cu) (net 3))
+  (segment (start 150.5 82) (end 151.772792 82) (width 0.75) (layer F.Cu) (net 3))
+  (segment (start 151.772792 82) (end 152.9 83.127208) (width 0.75) (layer F.Cu) (net 3))
+  (segment (start 152.9 83.127208) (end 152.9 88.24) (width 0.75) (layer F.Cu) (net 3))
+  (segment (start 152.9 88.24) (end 152.14 89) (width 0.75) (layer F.Cu) (net 3))
+  (segment (start 152.14 89) (end 150.54 89) (width 0.75) (layer F.Cu) (net 3))
+  (segment (start 150.54 92.5) (end 150.54 89) (width 0.75) (layer F.Cu) (net 3))
   (zone (net 0) (net_name "") (layer B.Cu) (hatch edge 0.508)
     (connect_pads (clearance 0.3))

Commit message: Fixups
Parts:
- moved RV1 2.00 mm to (145.4, 80.0)
- moved J1 1.00 mm to (150.5, 88.0)
- moved J2 0.50 mm to (150.5, 92.0)
Routing:
- net /VOL_1: track 20.6 -> 21.7 mm
- net /VOL_3: track 11.0 -> 12.0 mm
- net Net-(J1-Pad1): track 16.7 -> 16.1 mm

Commit message: Various
Parts:
- removed J2: Conn_01x03_Female, Pin_Headers:Pin_Header_Straight_1x03_Pitch2.54mm
- moved P1 4.50 mm to (147.0, 94.0)
- moved J1 0.50 mm to (150.5, 87.5)
Connections:
- J1 pad 1: Net-(J1-Pad1) -> Net-(C1-Pad1)
- RV1 pad 2: Net-(J1-Pad1) -> Net-(C1-Pad1)
- RV1 pad 3: Net-(J1-Pad1) -> Net-(RV1-Pad3)
Routing:
- net Net-(J1-Pad1): track 16.1 -> 0.00 mm
- net Net-(C1-Pad1): track 0.00 -> 14.5 mm
- net /VOL_1: track 21.7 -> 16.8 mm
- net /VOL_3: track 12.0 -> 7.98 mm
Other:
- board size 20 x 26 mm -> 12 x 21 mm
