File: BGP_MM/SW_BR/SW_BR.sch (KiCad schematic (older format))
At the start: 2 parts, among them P1 CONN_01X03, P2 CONN_01X02

Commit message: MM Refactoring
Parts:
- removed P1: CONN_01X03, LIBS:NKK_SPDT, symbol CONN_01X03
- added P1: CONN_01X04, Connectors_JST:JST_PH_B4B-PH-K_04x2.00mm_Straight, symbol CONN_01X04
- added P3: CONN_01X02, Connectors_JST:JST_PH_B2B-PH-K_02x2.00mm_Straight, symbol CONN_01X02
- added SW1: SW_DPDT, LIBS:NKK_DPDT, symbol SW_DPDT
Connections:
- net Earth: now also P1.1 (P1), P3.2 (P2), SW1.3 (C)
- net SEL_I: now reaches P2.1 (P1)
- net SEL_I: now also P1.3 (P3), SW1.6 (C)
- new net ACT_I: P1.2 (P2), SW1.4 (A)
- new net BR_I: P1.4 (P4), SW1.2 (B)
- new net VOL_O: P3.1 (P1), SW1.5 (B)
Other:
- note added: "To BT"
- note added: "To SEL"
- note added: "To VOL"
Changed lines of the file:
@@
 LIBS:contrib
 LIBS:valves
+LIBS:parts
 LIBS:SW_BR-cache
 EELAYER 25 0
@@
 $EndDescr
 $Comp
-L CONN_01X03 P1
-U 1 1 5B149C21
-P 5800 3800
-F 0 "P1" H 5800 4000 50  0000 C CNN
-F 1 "CONN_01X03" V 5900 3800 50  0001 C CNN
-F 2 "LIBS:NKK_SPDT" H 5800 3800 50  0001 C CNN
-F 3 "" H 5800 3800 50  0000 C CNN
-	1    5800 3800
-	-1   0    0    1
+L SW_DPDT SW1
+U 1 1 5B19C4A9
+P 4800 2300
+F 0 "SW1" H 4800 2470 50  0000 C CNN
+F 1 "SW_DPDT" H 4800 2100 50  0001 C CNN
+F 2 "LIBS:NKK_DPDT" H 4800 2300 50  0001 C CNN
+F 3 "" H 4800 2300 50  0001 C CNN
+	1    4800 2300
+	1    0    0    -1
 $EndComp
 $Comp
-L CONN_01X02 P2
-U 1 1 5B149C91
-P 6300 3850
-F 0 "P2" H 6300 3700 50  0000 C CNN
-F 1 "CONN_01X02" V 6400 3850 50  0001 C CNN
-F 2 "Connectors_JST:JST_PH_B2B-PH-K_02x2.00mm_Straight" H 6300 3850 50  0001 C CNN
-F 3 "" H 6300 3850 50  0000 C CNN
-	1    6300 3850
+L SW_DPDT SW1
+U 2 1 5B19C53A
+P 4800 2850
+F 0 "SW1" H 4800 3020 50  0000 C CNN
+F 1 "SW_DPDT" H 4800 2650 50  0001 C CNN
+F 2 "LIBS:NKK_DPDT" H 4800 2850 50  0001 C CNN
+F 3 "" H 4800 2850 50  0001 C CNN
+	2    4800 2850
 	1    0    0    -1
 $EndComp
-Wire Wire Line
-	6000 3700 6050 3700
-Wire Wire Line
-	6050 3700 6050 3950
+Text Label 4600 2850 2    60   ~ 0
+VOL_O
+Text Label 5000 2750 0    60   ~ 0
+ACT_I
+Text Label 5000 2950 0    60   ~ 0
+SEL_I
+Text Label 4600 2300 2    60   ~ 0
+BR_I
 $Comp
 L Earth #PWR01
-U 1 1 5B149F72
-P 6050 3950
-F 0 "#PWR01" H 6050 3700 50  0001 C CNN
-F 1 "Earth" H 6050 3800 50  0001 C CNN
-F 2 "" H 6050 3950 50  0000 C CNN
-F 3 "" H 6050 3950 50  0000 C CNN
-	1    6050 3950
+U 1 1 5B19C5E4
+P 5550 2200
+F 0 "#PWR01" H 5550 1950 50  0001 C CNN
+F 1 "Earth" H 5550 2050 50  0001 C CNN
+F 2 "" H 5550 2200 50  0000 C CNN
+F 3 "" H 5550 2200 50  0000 C CNN
+	1    5550 2200
+	0    1    1    0
+$EndComp
+Text Label 5550 2400 2    60   ~ 0
+SEL_I
+Text Label 5550 2300 2    60   ~ 0
+ACT_I
+Text Notes 5900 2200 0    60   ~ 0
+To BT
+$Comp
+L CONN_01X02 P2
+U 1 1 5B19C75B
+P 5750 2950
+F 0 "P2" H 5750 3100 50  0000 C CNN
+F 1 "CONN_01X02" V 5850 2950 50  0001 C CNN
+F 2 "Connectors_JST:JST_PH_B2B-PH-K_02x2.00mm_Straight" H 5750 2950 50  0001 C CNN
+F 3 "" H 5750 2950 50  0000 C CNN
+	1    5750 2950
 	1    0    0    -1
 $EndComp
-Wire Wire Line
-	6100 3800 6000 3800
-Wire Wire Line
-	6000 3900 6100 3900
-Connection ~ 6050 3900
+Text Notes 5900 2900 0    60   ~ 0
+To SEL
+Text Label 5550 2900 2    60   ~ 0
+SEL_I
+$Comp
+L Earth #PWR02
+U 1 1 5B19C7C6
+P 5550 3000
+F 0 "#PWR02" H 5550 2750 50  0001 C CNN
+F 1 "Earth" H 5550 2850 50  0001 C CNN
+F 2 "" H 5550 3000 50  0000 C CNN
+F 3 "" H 5550 3000 50  0000 C CNN
+	1    5550 3000
+	0    1    1    0
+$EndComp
+$Comp
+L CONN_01X02 P3
+U 1 1 5B19C7E0
+P 5750 3250
+F 0 "P3" H 5750 3400 50  0000 C CNN
+F 1 "CONN_01X02" V 5850 3250 50  0001 C CNN
+F 2 "Connectors_JST:JST_PH_B2B-PH-K_02x2.00mm_Straight" H 5750 3250 50  0001 C CNN
+F 3 "" H 5750 3250 50  0000 C CNN
+	1    5750 3250
+	1    0    0    -1
+$EndComp
+Text Notes 5900 3200 0    60   ~ 0
+To VOL
+$Comp
+L Earth #PWR03
+U 1 1 5B19C82F
+P 5550 3300
+F 0 "#PWR03" H 5550 3050 50  0001 C CNN
+F 1 "Earth" H 5550 3150 50  0001 C CNN
+F 2 "" H 5550 3300 50  0000 C CNN
+F 3 "" H 5550 3300 50  0000 C CNN
+	1    5550 3300
+	0    1    1    0
+$EndComp
+Text Label 5550 3200 2    60   ~ 0
+VOL_O
+Text Label 5550 2500 2    60   ~ 0
+BR_I
+$Comp
+L CONN_01X04 P1
+U 1 1 5B19C90C
+P 5750 2350
+F 0 "P1" H 5750 2600 50  0000 C CNN
+F 1 "CONN_01X04" V 5850 2350 50  0001 C CNN
+F 2 "Connectors_JST:JST_PH_B4B-PH-K_04x2.00mm_Straight" H 5750 2350 50  0001 C CNN
+F 3 "" H 5750 2350 50  0000 C CNN
+	1    5750 2350
+	1    0    0    -1
+$EndComp
+$Comp
+L Earth #PWR04
+U 1 1 5B19C971
+P 5000 2400
+F 0 "#PWR04" H 5000 2150 50  0001 C CNN
+F 1 "Earth" H 5000 2250 50  0001 C CNN
+F 2 "" H 5000 2400 50  0000 C CNN
+F 3 "" H 5000 2400 50  0000 C CNN
+	1    5000 2400
+	0    -1   -1   0
+$EndComp
 $EndSCHEMATC

Commit message: MM Refactoring
Parts:
- removed P1: CONN_01X04, Connectors_JST:JST_PH_B4B-PH-K_04x2.00mm_Straight, symbol CONN_01X04
- removed P2, P3: CONN_01X02, Connectors_JST:JST_PH_B2B-PH-K_02x2.00mm_Straight, symbol CONN_01X02
- added J1, J2, J3: Conn_01x05_Male, Pin_Headers:Pin_Header_Straight_1x05_Pitch2.54mm, symbol Conn_01x05_Male
- added J4: Conn_01x02, LIBS:TerminalBlock_Phoenix_MPT-2.54mm_2pol, symbol Conn_01x02
- added J5: Conn_01x03, LIBS:TerminalBlock_Phoenix_MPT-2.54mm_3pol, symbol Conn_01x03
Connections:
- net Earth: now also SW1.1 (A), J1.1 (Pin_1), J2.1 (Pin_1), J2.4 (Pin_4), J3.1 (Pin_1), J5.1 (Pin_1); no longer SW1.3 (C)
- net VOL_O: now also J2.2 (Pin_2), J5.2 (Pin_2); no longer SW1.5 (B)
- net ACT_I renamed MID
- net MID: now also J3.3 (Pin_3)
- net BR_I renamed BR
- net BR: now also J1.4 (Pin_4)
- net SEL_I renamed SEL
- net SEL: now also J1.3 (Pin_3), J2.5 (Pin_5)
- new net: J4.1 (Pin_1), J5.3 (Pin_3)
- new net ACT: J1.2 (Pin_2), J3.2 (Pin_2)
- new net VCC: J1.5 (Pin_5), J3.4 (Pin_4), J3.5 (Pin_5), J4.2 (Pin_2)
- new net VOL_I: J2.3 (Pin_3), SW1.5 (B)
Other:
- note added: "BAT"
- note added: "JACK"
- note added: "TO_MID\nJump 3 and 2 for bypass"
- moved on the sheet: SW1A, SW1B
