File: BGP_MM/SW_SEL/SW_SEL.sch (KiCad schematic (older format))
At the start: 4 parts, among them SW1 Switch_SPDT_x2

Commit message: MM Switch
Parts:
- removed J? (x2): Conn_01x02_Male, symbol Conn_01x02_Male
- added J1: CONN_01X03, Connectors_JST:JST_PH_B3B-PH-K_03x2.00mm_Straight, symbol CONN_01X03
- J2: renamed from J?; footprint (none) -> Connectors_JST:JST_PH_B2B-PH-K_02x2.00mm_Straight
Connections:
- net Earth: now also J1.1 (P1)
- net I_BR: now also J1.2 (P2)
- net I_NK: now also J1.3 (P3)
Changed lines of the file:
@@
 SIG_O
 $Comp
-L Earth #PWR?
+L Earth #PWR01
 U 1 1 5B074DFC
 P 5850 3500
-F 0 "#PWR?" H 5850 3250 50  0001 C CNN
+F 0 "#PWR01" H 5850 3250 50  0001 C CNN
 F 1 "Earth" H 5850 3350 50  0001 C CNN
 F 2 "" H 5850 3500 50  0000 C CNN
@@
 $EndComp
 $Comp
-L Earth #PWR?
+L Earth #PWR02
 U 1 1 5B074E3D
 P 5850 4150
-F 0 "#PWR?" H 5850 3900 50  0001 C CNN
+F 0 "#PWR02" H 5850 3900 50  0001 C CNN
 F 1 "Earth" H 5850 4000 50  0001 C CNN
 F 2 "" H 5850 4150 50  0000 C CNN
@@
 $EndComp
 $Comp
-L Conn_01x02_Male J?
-U 1 1 5B169C56
-P 6650 3500
-F 0 "J?" H 6650 3600 50  0000 C CNN
-F 1 "Conn_01x02_Male" H 6650 3300 50  0001 C CNN
-F 2 "" H 6650 3500 50  0001 C CNN
-F 3 "" H 6650 3500 50  0001 C CNN
-	1    6650 3500
-	-1   0    0    -1
-$EndComp
-$Comp
-L Conn_01x02_Male J?
-U 1 1 5B169CB9
-P 6650 3800
-F 0 "J?" H 6650 3900 50  0000 C CNN
-F 1 "Conn_01x02_Male" H 6650 3600 50  0001 C CNN
-F 2 "" H 6650 3800 50  0001 C CNN
-F 3 "" H 6650 3800 50  0001 C CNN
-	1    6650 3800
-	-1   0    0    -1
-$EndComp
-$Comp
-L Conn_01x02_Male J?
+L Conn_01x02_Male J2
 U 1 1 5B169CF7
 P 6650 4100
-F 0 "J?" H 6650 4200 50  0000 C CNN
+F 0 "J2" H 6650 4200 50  0000 C CNN
 F 1 "Conn_01x02_Male" H 6650 3900 50  0001 C CNN
-F 2 "" H 6650 4100 50  0001 C CNN
+F 2 "Connectors_JST:JST_PH_B2B-PH-K_02x2.00mm_Straight" H 6650 4100 50  0001 C CNN
 F 3 "" H 6650 4100 50  0001 C CNN
 	1    6650 4100
@@
 $EndComp
 $Comp
-L Earth #PWR?
+L Earth #PWR03
 U 1 1 5B169DEB
 P 6450 3500
-F 0 "#PWR?" H 6450 3250 50  0001 C CNN
+F 0 "#PWR03" H 6450 3250 50  0001 C CNN
 F 1 "Earth" H 6450 3350 50  0001 C CNN
 F 2 "" H 6450 3500 50  0000 C CNN
@@
 Text Label 6450 3600 2    60   ~ 0
 I_BR
-Text Label 6450 3900 2    60   ~ 0
+Text Label 6450 3700 2    60   ~ 0
 I_NK
 $Comp
-L Earth #PWR?
-U 1 1 5B169E27
-P 6450 3800
-F 0 "#PWR?" H 6450 3550 50  0001 C CNN
-F 1 "Earth" H 6450 3650 50  0001 C CNN
-F 2 "" H 6450 3800 50  0000 C CNN
-F 3 "" H 6450 3800 50  0000 C CNN
-	1    6450 3800
-	0    1    1    0
-$EndComp
-$Comp
-L Earth #PWR?
+L Earth #PWR04
 U 1 1 5B169E41
 P 6450 4100
-F 0 "#PWR?" H 6450 3850 50  0001 C CNN
+F 0 "#PWR04" H 6450 3850 50  0001 C CNN
 F 1 "Earth" H 6450 3950 50  0001 C CNN
 F 2 "" H 6450 4100 50  0000 C CNN
@@
 Text Label 6450 4200 2    60   ~ 0
 SIG_O
+$Comp
+L CONN_01X03 J1
+U 1 1 5B18CF0C
+P 6650 3600
+F 0 "J1" H 6650 3800 50  0000 C CNN
+F 1 "CONN_01X03" V 6750 3600 50  0000 C CNN
+F 2 "Connectors_JST:JST_PH_B3B-PH-K_03x2.00mm_Straight" H 6650 3600 50  0001 C CNN
+F 3 "" H 6650 3600 50  0000 C CNN
+	1    6650 3600
+	1    0    0    -1
+$EndComp
 $EndSCHEMATC

Commit message: MM Refactoring
Connections:
- net SIG_O renamed SEL_O
Changed lines of the file:
@@
 	5850 3700 5850 3950
 Text Label 5850 3700 0    60   ~ 0
-SIG_O
+SEL_O
 $Comp
 L Earth #PWR01
@@
 $EndComp
 Text Label 6450 4200 2    60   ~ 0
-SIG_O
+SEL_O
 $Comp
 L CONN_01X03 J1

Commit message: MM Refactoring
Parts:
- removed J1: CONN_01X03, Connectors_JST:JST_PH_B3B-PH-K_03x2.00mm_Straight, symbol CONN_01X03
- added J1: Conn_01x03_Male, Pin_Headers:Pin_Header_Straight_1x03_Pitch2.54mm, symbol Conn_01x03_Male
- J2: footprint Connectors_JST:JST_PH_B2B-PH-K_02x2.00mm_Straight -> Pin_Headers:Pin_Header_Straight_1x02_Pitch2.54mm
Connections:
- net Earth: now also J2.2 (Pin_2), J1.3 (Pin_3); no longer J2.1 (Pin_1)
- net I_BR: now also J1.2 (Pin_2)
- net I_NK: now also J1.1 (Pin_1)
- net SEL_O: now also J2.1 (Pin_1); no longer J2.2 (Pin_2)
Changed lines of the file:
@@
 F 0 "J2" H 6650 4200 50  0000 C CNN
 F 1 "Conn_01x02_Male" H 6650 3900 50  0001 C CNN
-F 2 "Connectors_JST:JST_PH_B2B-PH-K_02x2.00mm_Straight" H 6650 4100 50  0001 C CNN
+F 2 "Pin_Headers:Pin_Header_Straight_1x02_Pitch2.54mm" H 6650 4100 50  0001 C CNN
 F 3 "" H 6650 4100 50  0001 C CNN
 	1    6650 4100
@@
 L Earth #PWR04
 U 1 1 5B169E41
-P 6450 4100
-F 0 "#PWR04" H 6450 3850 50  0001 C CNN
-F 1 "Earth" H 6450 3950 50  0001 C CNN
-F 2 "" H 6450 4100 50  0000 C CNN
-F 3 "" H 6450 4100 50  0000 C CNN
-	1    6450 4100
+P 6450 4200
+F 0 "#PWR04" H 6450 3950 50  0001 C CNN
+F 1 "Earth" H 6450 4050 50  0001 C CNN
+F 2 "" H 6450 4200 50  0000 C CNN
+F 3 "" H 6450 4200 50  0000 C CNN
+	1    6450 4200
 	0    1    1    0
 $EndComp
-Text Label 6450 4200 2    60   ~ 0
+Text Label 6450 4100 2    60   ~ 0
 SEL_O
 $Comp
-L CONN_01X03 J1
-U 1 1 5B18CF0C
+L Conn_01x03_Male J1
+U 1 1 5B1B1C8C
 P 6650 3600
-F 0 "J1" H 6650 3800 50  0000 C CNN
-F 1 "CONN_01X03" V 6750 3600 50  0000 C CNN
-F 2 "Connectors_JST:JST_PH_B3B-PH-K_03x2.00mm_Straight" H 6650 3600 50  0001 C CNN
-F 3 "" H 6650 3600 50  0000 C CNN
+F 0 "J1" H 6650 3400 50  0000 C CNN
+F 1 "Conn_01x03_Male" H 6650 3400 50  0001 C CNN
+F 2 "Pin_Headers:Pin_Header_Straight_1x03_Pitch2.54mm" H 6650 3600 50  0001 C CNN
+F 3 "" H 6650 3600 50  0001 C CNN
 	1    6650 3600
-	1    0    0    -1
+	-1   0    0    1
 $EndComp
 $EndSCHEMATC
