File: BGP_MM/MID_STACK/MID_STACK.sch (KiCad schematic (older format))
At the start: 7 parts, among them P1 CONN_01X04, P2 CONN_01X09

Commit message: Updates MM
Parts:
- removed P1: CONN_01X04, Connectors_JST:JST_PH_B4B-PH-K_04x2.00mm_Straight, symbol CONN_01X04
- added J? (x3): Conn_01x02, symbol Conn_01x02
- added J? (x3): Conn_01x04_Male, symbol Conn_01x04_Male
- added J?: Conn_01x02_Male, symbol Conn_01x02_Male
- R3: value 100k -> 200k
Connections:
- net labels added: Earth, JZ_I, JZ_O, MM_BC, MM_BH, MM_I, MM_NC, MM_NH, MM_O, SIG_O
- wire segments 16 -> 17
Other:
- note added: "COIL SW"
- note added: "SELECT SW"
- note added: "To BT"
- note added: "To VOL"
- moved on the sheet: C1, C2, P2, R1, R2, R3

Commit message: MM Finished board layouts
Parts:
- removed J? (x3): Conn_01x02, symbol Conn_01x02
- added P2, P3: CONN_01X02, Terminal_Blocks:TerminalBlock_Pheonix_MPT-2.54mm_2pol, symbol CONN_01X02
- added P4: CONN_01X03, Terminal_Blocks:TerminalBlock_Pheonix_MPT-2.54mm_3pol, symbol CONN_01X03
- C1, C2: footprint Capacitor_THT:C_Rect_L7.2mm_W2.5mm_P5.00mm_FKS2_FKP2_MKS2_MKP2 -> Capacitor_THT:C_Rect_L4.6mm_W3.0mm_P2.50mm_MKS02_FKP02
- J1, J3, J4: renamed from J?; footprint (none) -> Connectors_JST:JST_PH_B4B-PH-K_04x2.00mm_Straight
- J2: renamed from J?; footprint (none) -> Connectors_JST:JST_PH_B2B-PH-K_02x2.00mm_Straight
- R2: renamed from R1; value 4.7k -> 10k
- R3: renamed from R2; value 4.7k -> 10k
- renumbered P2 to P1, R3 to R1
Connections:
- net labels removed: F1_1, F2_1, JZ_O, MM_O
Other:
- moved on the sheet: C1, C2, J1, J3, J4, P1, R1, R2, R3

Commit message: MM - Board changes
Parts:
- removed J2: Conn_01x02_Male, Connectors_JST:JST_PH_B2B-PH-K_02x2.00mm_Straight, symbol Conn_01x02_Male
- removed J3, J4: Conn_01x04_Male, Connectors_JST:JST_PH_B4B-PH-K_04x2.00mm_Straight, symbol Conn_01x04_Male
- removed P2, P3: CONN_01X02, Terminal_Blocks:TerminalBlock_Pheonix_MPT-2.54mm_2pol, symbol CONN_01X02
- removed P4: CONN_01X03, Terminal_Blocks:TerminalBlock_Pheonix_MPT-2.54mm_3pol, symbol CONN_01X03
- C1: footprint Capacitor_THT:C_Rect_L4.6mm_W3.0mm_P2.50mm_MKS02_FKP02 -> Capacitors_SMD:C_0805
- C2: footprint Capacitor_THT:C_Rect_L4.6mm_W3.0mm_P2.50mm_MKS02_FKP02 -> Capacitors_SMD:C_1206
Connections:
- net labels removed: Earth, JZ_I, MM_BC, MM_BH, MM_I, MM_NC, MM_NH, SIG_O
- wire segments 17 -> 15
Other:
- note removed: "COIL SW"
- note removed: "SELECT SW"
- note removed: "To VOL"
- moved on the sheet: C1, C2, J1, P1, R1, R2, R3

Commit message: tweaks
Connections:
- net MID_I: now also J1.1 (Pin_1); no longer J1.4 (Pin_4)
- net MID_O: now also J1.3 (Pin_3); no longer J1.2 (Pin_2)
- net MID_R: now also J1.2 (Pin_2); no longer J1.3 (Pin_3)
- net Vref: now also J1.4 (Pin_4); no longer J1.1 (Pin_1)
Changed lines of the file:
@@
 L Conn_01x04_Male J1
 U 1 1 5B03DCA0
-P 5000 3550
-F 0 "J1" H 5000 3750 50  0000 C CNN
-F 1 "Conn_01x04_Male" H 5000 3250 50  0001 C CNN
-F 2 "Connectors_JST:JST_PH_B4B-PH-K_04x2.00mm_Straight" H 5000 3550 50  0001 C CNN
-F 3 "" H 5000 3550 50  0001 C CNN
-	1    5000 3550
-	1    0    0    -1
+P 5000 3650
+F 0 "J1" H 5000 3850 50  0000 C CNN
+F 1 "Conn_01x04_Male" H 5000 3350 50  0001 C CNN
+F 2 "Connectors_JST:JST_PH_B4B-PH-K_04x2.00mm_Straight" H 5000 3650 50  0001 C CNN
+F 3 "" H 5000 3650 50  0001 C CNN
+	1    5000 3650
+	1    0    0    1
 $EndComp
 Text Label 7400 3950 2    60   ~ 0

Commit message: MM Gerbers Finished, Mid Stack Ammended J0
Parts:
- C1: footprint Capacitors_SMD:C_0805 -> Capacitors_SMD:C_1206
- C2: footprint Capacitors_SMD:C_1206 -> Capacitors_SMD:C_0805
Changed lines of the file:
@@
 F 0 "C1" H 6110 3820 50  0000 L CNN
 F 1 "22n" H 6110 3670 50  0000 L CNN
-F 2 "Capacitors_SMD:C_0805" H 6100 3750 50  0001 C CNN
+F 2 "Capacitors_SMD:C_1206" H 6100 3750 50  0001 C CNN
 F 3 "" H 6100 3750 50  0000 C CNN
 	1    6100 3750
@@
 F 0 "C2" H 6410 4520 50  0000 L CNN
 F 1 "10n" H 6410 4370 50  0000 L CNN
-F 2 "Capacitors_SMD:C_1206" H 6400 4450 50  0001 C CNN
+F 2 "Capacitors_SMD:C_0805" H 6400 4450 50  0001 C CNN
 F 3 "" H 6400 4450 50  0000 C CNN
 	1    6400 4450

Commit message: MM Refactoring
Parts:
- removed J1: Conn_01x04_Male, Connectors_JST:JST_PH_B4B-PH-K_04x2.00mm_Straight, symbol Conn_01x04_Male
- removed R1: 200k, Resistors_SMD:R_0603_HandSoldering, symbol R_Small
- added C3, C5, C6: 10u, Capacitors_SMD:C_0805, symbol CP1_Small
- added C4: 120p, Capacitors_SMD:C_0603_HandSoldering, symbol C_Small
- added P2, P3: CONN_01X02, Connectors_JST:JST_PH_B2B-PH-K_02x2.00mm_Straight, symbol CONN_01X02
- added R10, R4, R5, R9: 100k, Resistors_SMD:R_0603_HandSoldering, symbol R_Small
- added R3, R6: 20k, Resistors_SMD:R_0603_HandSoldering, symbol R_Small
- added R7: 1MEG, Resistors_SMD:R_0603_HandSoldering, symbol R_Small
- added R8: 1k, Resistors_SMD:R_0603_HandSoldering, symbol R_Small
- added U1: LM4250, Housings_SOIC:SOIC-8_3.9x4.9mm_Pitch1.27mm, symbol LM318N
- C1: value 22n -> 10n; footprint Capacitors_SMD:C_1206 -> Capacitors_SMD:C_0805
- C2: value 10n -> 4.7n
- renumbered R2 to R1, R3 to R2
Connections:
- net MID_I: now also C3.1, R3.1
- net MID_O: now also C4.1, R6.2, R8.1, U1.6
- net MID_R: now also U1.3 (+)
- net Vref: now also C5.1, R4.2, R5.1
- new net: C4.2, R3.2, R6.1, U1.2 (-)
- new net: C6.2, R8.2
- new net Earth: C5.2, P3.2 (P2), R10.2, R5.2, R7.1, R9.2, U1.4 (V-)
- new net IN: C3.2, P2.1 (P1), R10.1
- new net OUT: C6.1, P2.2 (P2), R9.1
- new net VCC: P3.1 (P1), R4.1, U1.7 (V+)
Other:
- note removed: "To BT"
- moved on the sheet: C1, C2, P1, R1, R2

Commit message: MM Refactoring
Parts:
- removed P2, P3: CONN_01X02, Connectors_JST:JST_PH_B2B-PH-K_02x2.00mm_Straight, symbol CONN_01X02
- removed R7: 1MEG, Resistors_SMD:R_0603_HandSoldering, symbol R_Small
- added J1: Conn_01x04_Male, Pin_Headers:Pin_Header_Straight_2x02_Pitch2.54mm, symbol Conn_01x04_Male
- U1: value LM4250 -> TL061
- renumbered P1 to RV1
Connections:
- net Earth: now also J1.4 (Pin_4)
- net IN: now also J1.2 (Pin_2)
- net OUT: now also C6.2, J1.1 (Pin_1); no longer C6.1
- net VCC: now also J1.3 (Pin_3)
- net at R8.2: now also C6.1; no longer C6.2
Changed lines of the file:
@@
 MID_R
 $Comp
-L CONN_01X09 P1
+L CONN_01X09 RV1
 U 1 1 5A669FB9
 P 4200 3400
-F 0 "P1" H 4200 3900 50  0000 C CNN
+F 0 "RV1" H 4200 3900 50  0000 C CNN
 F 1 "CONN_01X09" V 4300 3400 50  0001 C CNN
 F 2 "LIBS:Potentiometer_Alpha_Tripple_Vertical_Dual_Shaft" H 4200 3400 50  0001 C CNN
@@
 P 5850 3300
 F 0 "U1" H 5850 3600 50  0000 L CNN
-F 1 "LM4250" H 5850 3050 50  0000 L CNN
+F 1 "TL061" H 5850 3050 50  0000 L CNN
 F 2 "Housings_SOIC:SOIC-8_3.9x4.9mm_Pitch1.27mm" H 5850 3300 50  0001 C CNN
 F 3 "" H 5850 3300 50  0000 C CNN
@@
 F 3 "" H 6700 3300 50  0000 C CNN
 	1    6700 3300
-	0    1    1    0
+	0    -1   -1   0
 $EndComp
 $Comp
@@
 $EndComp
 $Comp
-L R_Small R7
-U 1 1 5B1A4567
-P 6200 3100
-F 0 "R7" H 6230 3120 50  0000 L CNN
-F 1 "1MEG" H 6230 3060 50  0000 L CNN
-F 2 "Resistors_SMD:R_0603_HandSoldering" H 6200 3100 50  0001 C CNN
-F 3 "" H 6200 3100 50  0000 C CNN
-	1    6200 3100
-	1    0    0    -1
-$EndComp
-$Comp
 L R_Small R3
 U 1 1 5B1A4626
@@
 	0    -1   -1   0
 $EndComp
-$Comp
-L Earth #PWR01
-U 1 1 5B1A4724
-P 6200 3000
-F 0 "#PWR01" H 6200 2750 50  0001 C CNN
-F 1 "Earth" H 6200 2850 50  0001 C CNN
-F 2 "" H 6200 3000 50  0000 C CNN
-F 3 "" H 6200 3000 50  0000 C CNN
-	1    6200 3000
-	-1   0    0    1
-$EndComp
-Wire Wire Line
-	6150 3200 6200 3200
-Wire Wire Line
-	6350 3300 6150 3300
+Wire Wire Line
+	6150 3300 6350 3300
 Wire Wire Line
 	6600 3300 6550 3300
 Wire Wire Line
-	5550 3400 5400 3400
+	5400 3400 5550 3400
 Wire Wire Line
 	5200 3400 5050 3400
@@
 MID_R
 $Comp
-L VCC #PWR02
+L VCC #PWR01
 U 1 1 5B1A4A30
 P 5750 3000
-F 0 "#PWR02" H 5750 2850 50  0001 C CNN
+F 0 "#PWR01" H 5750 2850 50  0001 C CNN
 F 1 "VCC" H 5750 3150 50  0000 C CNN
 F 2 "" H 5750 3000 50  0000 C CNN
@@
 $EndComp
 Wire Wire Line
-	5650 5100 5650 4950
+	5650 4950 5650 5100
 Wire Wire Line
 	5650 5050 5900 5050
@@
 Vref
 $Comp
-L Earth #PWR03
+L Earth #PWR02
 U 1 1 5B1A4F27
 P 5750 3600
-F 0 "#PWR03" H 5750 3350 50  0001 C CNN
+F 0 "#PWR02" H 5750 3350 50  0001 C CNN
 F 1 "Earth" H 5750 3450 50  0001 C CNN
 F 2 "" H 5750 3600 50  0000 C CNN
@@
 $EndComp
 $Comp
-L Earth #PWR04
+L Earth #PWR03
 U 1 1 5B1A4FE2
 P 5650 5350
-F 0 "#PWR04" H 5650 5100 50  0001 C CNN
+F 0 "#PWR03" H 5650 5100 50  0001 C CNN
 F 1 "Earth" H 5650 5200 50  0001 C CNN
 F 2 "" H 5650 5350 50  0000 C CNN
@@
 $EndComp
 $Comp
-L VCC #PWR05
+L VCC #PWR04
 U 1 1 5B1A506F
 P 5650 4750
-F 0 "#PWR05" H 5650 4600 50  0001 C CNN
+F 0 "#PWR04" H 5650 4600 50  0001 C CNN
 F 1 "VCC" H 5650 4900 50  0000 C CNN
 F 2 "" H 5650 4750 50  0000 C CNN
@@
 $EndComp
 $Comp
-L Earth #PWR06
+L Earth #PWR05
 U 1 1 5B1A569C
 P 6900 3650
-F 0 "#PWR06" H 6900 3400 50  0001 C CNN
+F 0 "#PWR05" H 6900 3400 50  0001 C CNN
 F 1 "Earth" H 6900 3500 50  0001 C CNN
 F 2 "" H 6900 3650 50  0000 C CNN
@@
 	6900 3300 6900 3400
 $Comp
-L VCC #PWR07
+L VCC #PWR06
 U 1 1 5B1A592E
-P 7550 3750
-F 0 "#PWR07" H 7550 3600 50  0001 C CNN
-F 1 "VCC" H 7550 3900 50  0000 C CNN
-F 2 "" H 7550 3750 50  0000 C CNN
-F 3 "" H 7550 3750 50  0000 C CNN
-	1    7550 3750
-	1    0    0    -1
-$EndComp
-$Comp
-L Earth #PWR08
+P 7550 3500
+F 0 "#PWR06" H 7550 3350 50  0001 C CNN
+F 1 "VCC" H 7550 3650 50  0000 C CNN
+F 2 "" H 7550 3500 50  0000 C CNN
+F 3 "" H 7550 3500 50  0000 C CNN
+	1    7550 3500
+	0    1    1    0
+$EndComp
+$Comp
+L Earth #PWR07
 U 1 1 5B1A5972
-P 7550 3850
-F 0 "#PWR08" H 7550 3600 50  0001 C CNN
-F 1 "Earth" H 7550 3700 50  0001 C CNN
-F 2 "" H 7550 3850 50  0000 C CNN
-F 3 "" H 7550 3850 50  0000 C CNN
-	1    7550 3850
+P 7550 3600
+F 0 "#PWR07" H 7550 3350 50  0001 C CNN
+F 1 "Earth" H 7550 3450 50  0001 C CNN
+F 2 "" H 7550 3600 50  0000 C CNN
+F 3 "" H 7550 3600 50  0000 C CNN
+	1    7550 3600
 	1    0    0    -1
 $EndComp
@@
 Text Label 6900 3300 0    60   ~ 0
 OUT
-Text Label 7550 3500 0    60   ~ 0
+Text Label 7550 3300 0    60   ~ 0
 OUT
 Text Label 7550 3400 0    60   ~ 0
@@
 $EndComp
 $Comp
-L Earth #PWR09
+L Earth #PWR08
 U 1 1 5B1A1AD5
 P 4750 3800
-F 0 "#PWR09" H 4750 3550 50  0001 C CNN
+F 0 "#PWR08" H 4750 3550 50  0001 C CNN
 F 1 "Earth" H 4750 3650 50  0001 C CNN
 F 2 "" H 4750 3800 50  0000 C CNN
@@
 	4750 3400 4850 3400
 $Comp
-L CONN_01X02 P2
-U 1 1 5B1A36D9
-P 7350 3450
-F 0 "P2" H 7350 3600 50  0000 C CNN
-F 1 "CONN_01X02" V 7450 3450 50  0001 C CNN
-F 2 "Connectors_JST:JST_PH_B2B-PH-K_02x2.00mm_Straight" H 7350 3450 50  0001 C CNN
-F 3 "" H 7350 3450 50  0000 C CNN
-	1    7350 3450
-	-1   0    0    -1
-$EndComp
-$Comp
-L CONN_01X02 P3
-U 1 1 5B1A37B9
-P 7350 3800
-F 0 "P3" H 7350 3950 50  0000 C CNN
-F 1 "CONN_01X02" V 7450 3800 50  0001 C CNN
-F 2 "Connectors_JST:JST_PH_B2B-PH-K_02x2.00mm_Straight" H 7350 3800 50  0001 C CNN
-F 3 "" H 7350 3800 50  0000 C CNN
-	1    7350 3800
-	-1   0    0    -1
+L Conn_01x04_Male J1
+U 1 1 5B1AEF93
+P 7350 3400
+F 0 "J1" H 7350 3600 50  0000 C CNN
+F 1 "Conn_01x04_Male" H 7350 3100 50  0001 C CNN
+F 2 "Pin_Headers:Pin_Header_Straight_2x02_Pitch2.54mm" H 7350 3400 50  0001 C CNN
+F 3 "" H 7350 3400 50  0001 C CNN
+	1    7350 3400
+	1    0    0    -1
 $EndComp
 $EndSCHEMATC

Commit message: Minor tweaks for MM/F0 - gerbers ready to go out
Parts:
- U1: symbol LM318N -> LM318N-RESCUE-MID_STACK
Changed lines of the file:
@@
 EESchema Schematic File Version 2
+LIBS:MID_STACK-rescue
 LIBS:power
 LIBS:device
@@
 MID_R
 $Comp
-L LM318N U1
+L LM318N-RESCUE-MID_STACK U1
 U 1 1 5B1A4170
 P 5850 3300
