File: BGP_F0/BT_STACK_v1.1/BT_STACK.kicad_pcb (KiCad board)
At the start: 2 copper layers, 24 x 26 mm, 20 parts, among them P1 CONN_01X05, P2 CONN_01X02, P3 CONN_01X04, U1 MC33178

Commit message: F0 Gerbers
Parts:
- moved P2 2.59 mm to (143.2, 73.3)
- moved RV1 2.00 mm to (148.2, 73.5)
- moved C6 1.90 mm to (143.8, 88.9)
- moved R4 1.90 mm to (144.0, 78.4)
- moved R5 1.90 mm to (144.0, 80.9)
- moved R6 1.90 mm to (144.0, 83.4)
- moved R8 1.90 mm to (144.0, 86.4)
- moved C5 1.30 mm to (160.3, 73.3)
- moved P1 0.85 mm to (143.0, 91.5)
- moved P3 0.85 mm to (155.0, 91.5)
- moved C3 0.30 mm to (160.0, 84.0)
Routing:
- net /B+: track 28.2 -> 23.1 mm
- net Earth: track 26.9 -> 22.4 mm
- net Net-(C6-Pad2): track 25.2 -> 29.1 mm
- net /TW: track 12.3 -> 9.03 mm
- net /T+: track 6.20 -> 3.36 mm
- net /IN: track 31.1 -> 28.8 mm
- net /MID_R: track 19.9 -> 18.3 mm
- net /BW: track 25.7 -> 24.3 mm, vias 1 -> 0
- net /B-: track 19.6 -> 18.5 mm
- net /MID_I: track 34.4 -> 33.5 mm
- net Net-(C2-Pad1): track 14.4 -> 15.2 mm
- net /V+: track 11.2 -> 10.4 mm
- net /T-: track 4.80 -> 4.14 mm
Other:
- board size 24 x 26 mm -> 22 x 23 mm

Commit message: Minor tweaks for MM/F0 - gerbers ready to go out
Parts:
- P1: footprint Connectors_JST:JST_PH_B5B-PH-K_05x2.00mm_Straight -> Pin_Headers:Pin_Header_Straight_1x05
- P3: value CONN_01X04 -> CONN_01X05; footprint Connectors_JST:JST_PH_B4B-PH-K_04x2.00mm_Straight -> Pin_Headers:Pin_Header_Straight_1x05
- moved P3 8.10 mm to (146.9, 91.0), turned to 270 degrees
- moved P1 4.76 mm to (146.9, 94.2), turned to 270 degrees
- moved C6 0.91 mm to (143.9, 88.0)
- moved R8 0.90 mm to (144.0, 85.5)
Routing:
- net /IN: track 28.8 -> 22.8 mm
- net Earth: track 22.4 -> 27.4 mm
- net /V+: track 10.4 -> 13.5 mm, vias 0 -> 1
- net /MID_O: track 23.0 -> 20.2 mm
- net /MID_I: track 33.5 -> 30.8 mm, vias 0 -> 1
- net /MID_R: track 18.3 -> 17.2 mm, vias 1 -> 0
- net /OUT: track 7.27 -> 8.01 mm
- net Net-(C6-Pad2): track 29.1 -> 28.4 mm
Other:
- board size 22 x 23 mm -> 22 x 25 mm
- net class Default: clearance 0.3 -> 0.25
- net class PWR: clearance 0.3 -> 0.25; trace_width 0.5 -> 0.3
- rule trace_clearance: 0.3 -> 0.25
- rule trace_min: 0.3 -> 0.25

Commit message: BOM Work prior to sending Gerbers
Parts:
- C1: value 22u -> 10u; footprint Capacitors_SMD:C_0805_HandSoldering -> Capacitors_SMD:C_1206_HandSoldering
- C2: footprint Capacitors_Tantalum_SMD:TantalC_SizeR_EIA-2012 -> Capacitors_SMD:C_0805_HandSoldering
- moved C1 1.25 mm to (147.0, 87.0)
- turned C2 to 180 degrees
Routing:
- net /V+: track 13.5 -> 10.3 mm
- net /MID_O: track 20.2 -> 19.1 mm
Changed lines of the file:
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@@
     (links 38)
     (no_connects 0)
-    (area 140.05 68.914286 163.075001 97.35)
+    (area 140.924999 70.924999 163.075001 96.075001)
     (thickness 1.6)
     (drawings 8)
@@
     )
   )
-  (module Capacitors_SMD:C_0805_HandSoldering (layer B.Cu)
-    (at 145.75 87 180)
-    (descr "Capacitor SMD 0805, hand soldering")
-    (tags "capacitor 0805")
-    (attr smd)
-    (fp_text reference C1 (at 1.8 -1.4 180) (layer B.SilkS)
-      (effects (font (size 0.6 0.6) (thickness 0.15)) (justify mirror))
-    )
-    (fp_text value 22u (at 0 -2.1 180) (layer B.Fab) hide
-      (effects (font (size 0.6 0.6) (thickness 0.15)) (justify mirror))
-    )
-    (fp_line (start -2.3 1) (end 2.3 1) (layer B.CrtYd) (width 0.05))
-    (fp_line (start -2.3 -1) (end 2.3 -1) (layer B.CrtYd) (width 0.05))
-    (fp_line (start -2.3 1) (end -2.3 -1) (layer B.CrtYd) (width 0.05))
-    (fp_line (start 2.3 1) (end 2.3 -1) (layer B.CrtYd) (width 0.05))
-    (fp_line (start 0.5 0.85) (end -0.5 0.85) (layer B.SilkS) (width 0.15))
-    (fp_line (start -0.5 -0.85) (end 0.5 -0.85) (layer B.SilkS) (width 0.15))
-    (pad 1 smd rect (at -1.25 0 180) (size 1.5 1.25) (layers B.Cu B.Paste B.Mask)
-      (net 1 /V+))
-    (pad 2 smd rect (at 1.25 0 180) (size 1.5 1.25) (layers B.Cu B.Paste B.Mask)
-      (net 2 Earth))
-    (model Capacitors_SMD.3dshapes/C_0805_HandSoldering.wrl
-      (at (xyz 0 0 0))
-      (scale (xyz 1 1 1))
-      (rotate (xyz 0 0 0))
-    )
-  )
   (module Resistors_SMD:R_0603_HandSoldering (layer F.Cu)
     (at 144 83.4)
@@
     )
   )
-  (module Capacitors_Tantalum_SMD:TantalC_SizeR_EIA-2012 (layer B.Cu)
-    (at 154 87)
-    (descr "Tantal Cap. , Size C, EIA-2012")
-    (fp_text reference C2 (at 1.6 -1.6) (layer B.SilkS)
-      (effects (font (size 0.6 0.6) (thickness 0.15)) (justify mirror))
-    )
-    (fp_text value 10u (at 0 -1.27) (layer B.Fab) hide
-      (effects (font (size 0.6 0.6) (thickness 0.15)) (justify mirror))
-    )
-    (fp_line (start 0.635 0.635) (end 0.635 -0.635) (layer B.SilkS) (width 0.15))
-    (fp_line (start -1.016 0.635) (end -1.016 -0.635) (layer B.SilkS) (width 0.15))
-    (fp_line (start -1.016 -0.635) (end 1.016 -0.635) (layer B.SilkS) (width 0.15))
-    (fp_line (start 1.016 -0.635) (end 1.016 0.635) (layer B.SilkS) (width 0.15))
-    (fp_line (start 1.016 0.635) (end -1.016 0.635) (layer B.SilkS) (width 0.15))
-    (pad 1 smd rect (at 1.17602 0) (size 1.5494 1.80086) (layers B.Cu B.Paste B.Mask)
-      (net 17 "Net-(C2-Pad1)"))
-    (pad 2 smd rect (at -1.17602 0) (size 1.5494 1.80086) (layers B.Cu B.Paste B.Mask)
-      (net 4 /OUT))
-    (model Capacitors_Tantalum_SMD.3dshapes/TantalC_SizeR_EIA-2012.wrl
-      (at (xyz 0 0 0))
-      (scale (xyz 1 1 1))
-      (rotate (xyz 0 0 0))
-    )
-  )
   (module Capacitors_SMD:C_0805_HandSoldering (layer F.Cu)
     (at 160.3 73.3)
@@
     )
   )
+  (module Capacitors_SMD:C_1206_HandSoldering (layer B.Cu)
+    (at 147 87 180)
+    (descr "Capacitor SMD 1206, hand soldering")
+    (tags "capacitor 1206")
+    (attr smd)
+    (fp_text reference C1 (at 0 1.475001 180) (layer B.SilkS)
+      (effects (font (size 0.6 0.6) (thickness 0.15)) (justify mirror))
+    )
+    (fp_text value 10u (at 0 -2.3 180) (layer B.Fab)
+      (effects (font (size 0.6 0.6) (thickness 0.15)) (justify mirror))
+    )
+    (fp_line (start -3.3 1.15) (end 3.3 1.15) (layer B.CrtYd) (width 0.05))
+    (fp_line (start -3.3 -1.15) (end 3.3 -1.15) (layer B.CrtYd) (width 0.05))
+    (fp_line (start -3.3 1.15) (end -3.3 -1.15) (layer B.CrtYd) (width 0.05))
+    (fp_line (start 3.3 1.15) (end 3.3 -1.15) (layer B.CrtYd) (width 0.05))
+    (fp_line (start 1 1.025) (end -1 1.025) (layer B.SilkS) (width 0.15))
+    (fp_line (start -1 -1.025) (end 1 -1.025) (layer B.SilkS) (width 0.15))
+    (pad 1 smd rect (at -2 0 180) (size 2 1.6) (layers B.Cu B.Paste B.Mask)
+      (net 1 /V+))
+    (pad 2 smd rect (at 2 0 180) (size 2 1.6) (layers B.Cu B.Paste B.Mask)
+      (net 2 Earth))
+    (model Capacitors_SMD.3dshapes/C_1206_HandSoldering.wrl
+      (at (xyz 0 0 0))
+      (scale (xyz 1 1 1))
+      (rotate (xyz 0 0 0))
+    )
+  )
+  (module Capacitors_SMD:C_0805_HandSoldering (layer B.Cu)
+    (at 154 87 180)
+    (descr "Capacitor SMD 0805, hand soldering")
+    (tags "capacitor 0805")
+    (attr smd)
+    (fp_text reference C2 (at 0 1.275001 180) (layer B.SilkS)
+      (effects (font (size 0.6 0.6) (thickness 0.15)) (justify mirror))
+    )
+    (fp_text value 10u (at 0 -2.1 180) (layer B.Fab)
+      (effects (font (size 0.6 0.6) (thickness 0.15)) (justify mirror))
+    )
+    (fp_line (start -2.3 1) (end 2.3 1) (layer B.CrtYd) (width 0.05))
+    (fp_line (start -2.3 -1) (end 2.3 -1) (layer B.CrtYd) (width 0.05))
+    (fp_line (start -2.3 1) (end -2.3 -1) (layer B.CrtYd) (width 0.05))
+    (fp_line (start 2.3 1) (end 2.3 -1) (layer B.CrtYd) (width 0.05))
+    (fp_line (start 0.5 0.85) (end -0.5 0.85) (layer B.SilkS) (width 0.15))
+    (fp_line (start -0.5 -0.85) (end 0.5 -0.85) (layer B.SilkS) (width 0.15))
+    (pad 1 smd rect (at -1.25 0 180) (size 1.5 1.25) (layers B.Cu B.Paste B.Mask)
+      (net 17 "Net-(C2-Pad1)"))
+    (pad 2 smd rect (at 1.25 0 180) (size 1.5 1.25) (layers B.Cu B.Paste B.Mask)
+      (net 4 /OUT))
+    (model Capacitors_SMD.3dshapes/C_0805_HandSoldering.wrl
+      (at (xyz 0 0 0))
+      (scale (xyz 1 1 1))
+      (rotate (xyz 0 0 0))
+    )
+  )
   (gr_line (start 141 96) (end 163 96) (layer Edge.Cuts) (width 0.15))
   (gr_line (start 141.3 95.7) (end 162.7 95.7) (layer Margin) (width 0.2))
@@
   (gr_line (start 163 96) (end 163 71) (layer Edge.Cuts) (width 0.15))
   (gr_line (start 163 71) (end 141 71) (layer Edge.Cuts) (width 0.15))
-  (segment (start 152 94.2) (end 150.73639 92.93639) (width 0.3) (layer B.Cu) (net 1))
-  (segment (start 150.73639 92.93639) (end 150.73639 90.13639) (width 0.3) (layer B.Cu) (net 1))
-  (segment (start 150.73639 90.13639) (end 149.8 89.2) (width 0.3) (layer B.Cu) (net 1))
-  (segment (start 149.8 89.2) (end 148.05 89.2) (width 0.3) (layer B.Cu) (net 1))
-  (segment (start 148.05 89.2) (end 147 88.15) (width 0.3) (layer B.Cu) (net 1))
-  (segment (start 149.3 87.905) (end 147.245 87.905) (width 0.3) (layer F.Cu) (net 1))
-  (segment (start 147.245 87.905) (end 147 88.15) (width 0.3) (layer F.Cu) (net 1))
-  (via (at 147 88.15) (size 0.6) (drill 0.4) (layers F.Cu B.Cu) (net 1))
-  (segment (start 147 88.15) (end 147 87) (width 0.3) (layer B.Cu) (net 1))
+  (segment (start 150.1 89.3) (end 149 88.2) (width 0.3) (layer B.Cu) (net 1))
+  (segment (start 149 88.2) (end 149 87) (width 0.3) (layer B.Cu) (net 1))
+  (segment (start 150.73639 89.93639) (end 150.399999 89.599999) (width 0.3) (layer B.Cu) (net 1))
+  (segment (start 150.73639 92.78399) (end 150.73639 89.93639) (width 0.3) (layer B.Cu) (net 1))
+  (segment (start 149.3 87.905) (end 149.3 88.505) (width 0.3) (layer F.Cu) (net 1))
+  (segment (start 149.3 88.505) (end 150.095 89.3) (width 0.3) (layer F.Cu) (net 1))
+  (via (at 150.1 89.3) (size 0.6) (drill 0.4) (layers F.Cu B.Cu) (net 1))
+  (segment (start 152 94.0476) (end 150.73639 92.78399) (width 0.3) (layer B.Cu) (net 1))
+  (segment (start 150.095 89.3) (end 150.1 89.3) (width 0.3) (layer F.Cu) (net 1))
+  (segment (start 150.399999 89.599999) (end 150.1 89.3) (width 0.3) (layer B.Cu) (net 1))
+  (segment (start 152 94.2) (end 152 94.0476) (width 0.3) (layer B.Cu) (net 1))
   (segment (start 152 94.05) (end 152 94.2) (width 0.3) (layer B.Cu) (net 1))
-  (segment (start 152 94.2) (end 152 94.0476) (width 0.3) (layer B.Cu) (net 1))
-  (segment (start 148.825 87.905) (end 149.3 87.905) (width 0.3) (layer F.Cu) (net 1))
   (segment (start 146.92 94.2) (end 145.8064 94.2) (width 0.5) (layer B.Cu) (net 2))
   (segment (start 145.8064 94.2) (end 143 91.3936) (width 0.5) (layer B.Cu) (net 2))
@@
   (segment (start 144.5 87) (end 143.45 87) (width 0.5) (layer B.Cu) (net 2))
   (segment (start 143.45 87) (end 143 87) (width 0.5) (layer B.Cu) (net 2))
+  (segment (start 145.8 88) (end 144.9 88) (width 0.3) (layer F.Cu) (net 3))
+  (segment (start 149.46 90.8476) (end 148.2964 89.684) (width 0.3) (layer F.Cu) (net 3))
+  (segment (start 148.2964 89.684) (end 148.144 89.684) (width 0.3) (layer F.Cu) (net 3))
+  (segment (start 148.144 89.684) (end 146.46 88) (width 0.3) (layer F.Cu) (net 3))
+  (segment (start 146.46 88) (end 145.8 88) (width 0.3) (layer F.Cu) (net 3))
+  (segment (start 149.46 91) (end 149.46 90.8476) (width 0.3) (layer F.Cu) (net 3))
   (segment (start 144.9 88) (end 144.9 86.6) (width 0.3) (layer F.Cu) (net 3))
   (segment (start 144.9 86.6) (end 144.9 85.7) (width 0.3) (layer F.Cu) (net 3))
@@
   (segment (start 144.935 86.635) (end 144.9 86.6) (width 0.3) (layer F.Cu) (net 3))
   (segment (start 144.9 85.7) (end 145.1 85.5) (width 0.3) (layer F.Cu) (net 3))
-  (segment (start 145.4 89.2) (end 144.9 88.7) (width 0.3) (layer F.Cu) (net 3))
-  (segment (start 144.9 88.7) (end 144.9 88) (width 0.3) (layer F.Cu) (net 3))
-  (segment (start 148.926 89.2) (end 145.4 89.2) (width 0.3) (layer F.Cu) (net 3))
-  (segment (start 149.46 91) (end 149.46 89.734) (width 0.3) (layer F.Cu) (net 3))
-  (segment (start 149.46 89.734) (end 148.926 89.2) (width 0.3) (layer F.Cu) (net 3))
   (segment (start 149.3 86.635) (end 146.7 86.635) (width 0.3) (layer F.Cu) (net 3))
   (segment (start 146.7 84.05) (end 146.7 86.635) (width 0.3) (layer F.Cu) (net 3))
@@
   (segment (start 153.27 92.92) (end 154.54 94.19) (width 0.3) (layer B.Cu) (net 4))
   (segment (start 154.54 94.19) (end 154.54 94.2) (width 0.3) (layer B.Cu) (net 4))
-  (segment (start 153.2 87) (end 153.27 87.07) (width 0.3) (layer B.Cu) (net 4))
   (segment (start 157.099993 83.599999) (end 156.799994 83.3) (width 0.3) (layer F.Cu) (net 5))
   (segment (start 157.499994 84) (end 157.099993 83.599999) (width 0.3) (layer F.Cu) (net 5))

Commit message: BOM Updates
Parts:
- R9: value 100k -> 200k
Changed lines of the file:
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@@
-(kicad_pcb (version 4) (host pcbnew 4.0.4-1.fc24-product)
+(kicad_pcb (version 4) (host pcbnew 4.0.7)
   (general
     (links 38)
@@
       (effects (font (size 0.6 0.6) (thickness 0.15)))
     )
-    (fp_text value 100k (at 0 1.9) (layer F.Fab) hide
+    (fp_text value 200k (at 0 1.9) (layer F.Fab) hide
       (effects (font (size 0.6 0.6) (thickness 0.15)))
     )
