File: BGP_F0/BT_STACK_v1.1/BT_STACK.sch (KiCad schematic (older format))
At the start: 20 parts, among them P1 CONN_01X05, P2 CONN_01X02, P3 CONN_01X04, U1 MC33178

Commit message: Minor tweaks for MM/F0 - gerbers ready to go out
Parts:
- removed P3: CONN_01X04, Connectors_JST:JST_PH_B4B-PH-K_04x2.00mm_Straight, symbol CONN_01X04
- added P3: CONN_01X05, Pin_Headers:Pin_Header_Straight_1x05, symbol CONN_01X05
- P1: footprint Connectors_JST:JST_PH_B5B-PH-K_05x2.00mm_Straight -> Pin_Headers:Pin_Header_Straight_1x05
Connections:
- net MID_I: now also P3.4 (P4)
- net MID_O: now also P3.2 (P2)
- net MID_R: now also P3.3 (P3)
- net Vref: now also P3.1 (P1)
Changed lines of the file:
@@
 F 0 "P1" H 3750 2800 50  0000 C CNN
 F 1 "CONN_01X05" V 3850 2500 50  0000 C CNN
-F 2 "Connectors_JST:JST_PH_B5B-PH-K_05x2.00mm_Straight" H 3750 2500 50  0001 C CNN
+F 2 "Pin_Headers:Pin_Header_Straight_1x05" H 3750 2500 50  0001 C CNN
 F 3 "" H 3750 2500 50  0000 C CNN
 	1    3750 2500
@@
 $EndComp
 $Comp
-L Earth #PWR01
+L Earth #PWR1
 U 1 1 5A5AEE2D
 P 3950 2700
-F 0 "#PWR01" H 3950 2450 50  0001 C CNN
+F 0 "#PWR1" H 3950 2450 50  0001 C CNN
 F 1 "Earth" H 3950 2550 50  0001 C CNN
 F 2 "" H 3950 2700 50  0001 C CNN
@@
 Vref
 $Comp
-L Earth #PWR02
+L Earth #PWR2
 U 1 1 5A66674C
 P 4400 2600
-F 0 "#PWR02" H 4400 2350 50  0001 C CNN
+F 0 "#PWR2" H 4400 2350 50  0001 C CNN
 F 1 "Earth" H 4400 2450 50  0001 C CNN
 F 2 "" H 4400 2600 50  0001 C CNN
@@
 $EndComp
 $Comp
-L Earth #PWR03
+L Earth #PWR3
 U 1 1 5A666795
 P 5300 3000
-F 0 "#PWR03" H 5300 2750 50  0001 C CNN
+F 0 "#PWR3" H 5300 2750 50  0001 C CNN
 F 1 "Earth" H 5300 2850 50  0001 C CNN
 F 2 "" H 5300 3000 50  0001 C CNN
@@
 V+
 $Comp
-L Earth #PWR04
+L Earth #PWR4
 U 1 1 5A666848
 P 7100 3000
-F 0 "#PWR04" H 7100 2750 50  0001 C CNN
+F 0 "#PWR4" H 7100 2750 50  0001 C CNN
 F 1 "Earth" H 7100 2850 50  0001 C CNN
 F 2 "" H 7100 3000 50  0001 C CNN
@@
 Text Label 6900 2600 3    60   ~ 0
 MID_R
-$Comp
-L CONN_01X04 P3
-U 1 1 5A667029
-P 8800 2450
-F 0 "P3" H 8800 2700 50  0000 C CNN
-F 1 "CONN_01X04" V 8900 2450 50  0000 C CNN
-F 2 "Connectors_JST:JST_PH_B4B-PH-K_04x2.00mm_Straight" H 8800 2450 50  0001 C CNN
-F 3 "" H 8800 2450 50  0000 C CNN
-	1    8800 2450
-	1    0    0    -1
-$EndComp
 Text Label 8600 2300 2    60   ~ 0
 Vref
@@
 Text Label 4850 5000 0    60   ~ 0
 BW
+$Comp
+L CONN_01X05 P3
+U 1 1 5B1F5F6B
+P 8800 2500
+F 0 "P3" H 8800 2800 50  0000 C CNN
+F 1 "CONN_01X05" V 8900 2500 50  0000 C CNN
+F 2 "Pin_Headers:Pin_Header_Straight_1x05" H 8800 2500 50  0001 C CNN
+F 3 "" H 8800 2500 50  0000 C CNN
+	1    8800 2500
+	1    0    0    -1
+$EndComp
 $EndSCHEMATC

Commit message: BOM Work prior to sending Gerbers
Parts:
- C1: value 22u -> 10u; footprint Capacitors_SMD:C_0805_HandSoldering -> Capacitors_SMD:C_1206_HandSoldering
- C2: footprint Capacitors_Tantalum_SMD:TantalC_SizeR_EIA-2012 -> Capacitors_SMD:C_0805_HandSoldering
Other:
- moved on the sheet: C1, C2, C3, C4, C5, C6, P1, P2, P3, R1, R2, R3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

Commit message: BOM Updates
Parts:
- R9: value 100k -> 200k
Changed lines of the file:
@@
 P 6450 3050
 F 0 "R9" H 6480 3070 50  0000 L CNN
-F 1 "100k" H 6480 3010 50  0000 L CNN
+F 1 "200k" H 6480 3010 50  0000 L CNN
 F 2 "Resistors_SMD:R_0603_HandSoldering" H 6450 3050 50  0001 C CNN
 F 3 "" H 6450 3050 50  0000 C CNN
